File: wallputer/wallputer.kicad_pcb (KiCad board)
At the start: 2 copper layers, 244 parts, among them J1 For ROM uploading and control, J2 DE9_Socket, J3 4x20 character display, Q1 BS250, Q2 2N7000, Q3 BS250, Q4 2N7000, Q5 BS170, Q6 BS170, Q7 BC547, SW1 Reset, SW2 step, SW3 switch clock, U1 W65C02SxP, U10 MAX232, U11 NE555P, U12 74HC04, U13 NE555P, U14 74HC14, U15 74HC93, U16 74HC04, U17 74HC04, U18 74HC04, U19 74HC04, U2 SST39SF010, U21 SST39SF010, U22 INND-TS40, U23 INND-TS40, U24 SST39SF010, U25 INND-TS40, U26 INND-TS40, U27 SST39SF010, U28 INND-TS40, U29 INND-TS40, U3 HM62256BLP, U32 NE555P, U4 74HC00, U5 74HC153, U6 W65C51NxP, U7 W65C22SxP, U8 74HC00, Y2 1.8432Mhz, Y3 1 MHz

Commit message: more components routed
Parts:
- removed D38, D39: D, Diode_THT:D_5KPW_P12.70mm_Horizontal
- added C15: 1000uF, Capacitor_THT:CP_Axial_L20.0mm_D10.0mm_P26.00mm_Horizontal, F.Cu at (18.4, 361.0)
- added C16: 100nF, Capacitor_THT:C_Disc_D5.0mm_W2.5mm_P5.00mm, F.Cu at (191.1, 260.4)
- added C17: 100nF, Capacitor_THT:C_Disc_D5.0mm_W2.5mm_P5.00mm, F.Cu at (199.3, 347.3)
- added C18: 100nF, Capacitor_THT:C_Disc_D5.0mm_W2.5mm_P5.00mm, F.Cu at (59.6, 261.6)
- added C19: 100nF, Capacitor_THT:C_Disc_D5.0mm_W2.5mm_P5.00mm, F.Cu at (236.2, 347.3)
- added C20: 100nF, Capacitor_THT:C_Disc_D5.0mm_W2.5mm_P5.00mm, F.Cu at (330.5, 347.4)
- added C21: 100nF, Capacitor_THT:C_Disc_D5.0mm_W2.5mm_P5.00mm, F.Cu at (264.8, 347.3)
- added C22: 100nF, Capacitor_THT:C_Disc_D5.0mm_W2.5mm_P5.00mm, F.Cu at (293.4, 347.3)
- added C23: 100nF, Capacitor_THT:C_Disc_D5.0mm_W2.5mm_P5.00mm, F.Cu at (214.6, 260.4)
- added C24: 100nF, Capacitor_THT:C_Disc_D5.0mm_W2.5mm_P5.00mm, F.Cu at (170.9, 370.8)
- added C25: 100nF, Capacitor_THT:C_Disc_D5.0mm_W2.5mm_P5.00mm, F.Cu at (393.2, 171.6)
- added C26: 100nF, Capacitor_THT:C_Disc_D5.0mm_W2.5mm_P5.00mm, F.Cu at (116.8, 260.5)
- added C27: 100nF, Capacitor_THT:C_Disc_D5.0mm_W2.5mm_P5.00mm, F.Cu at (151.8, 260.4)
- added C28: 100nF, Capacitor_THT:C_Disc_D5.0mm_W2.5mm_P5.00mm, F.Cu at (31.1, 264.2)
- added C29: 100nF, Capacitor_THT:C_Disc_D5.0mm_W2.5mm_P5.00mm, F.Cu at (45.8, 233.0)
- added C30: 100nF, Capacitor_THT:C_Disc_D5.0mm_W2.5mm_P5.00mm, F.Cu at (87.7, 229.2)
- added C31: 100nF, Capacitor_THT:C_Disc_D5.0mm_W2.5mm_P5.00mm, F.Cu at (43.8, 261.6)
- added C32: 100nF, Capacitor_THT:C_Disc_D5.0mm_W2.5mm_P5.00mm, F.Cu at (401.4, 167.6)
- added C33: 100nF, Capacitor_THT:C_Disc_D5.0mm_W2.5mm_P5.00mm, F.Cu at (401.4, 171.6)
- added C34: 100nF, Capacitor_THT:C_Disc_D5.0mm_W2.5mm_P5.00mm, F.Cu at (401.4, 175.7)
- added C35: 100nF, Capacitor_THT:C_Disc_D5.0mm_W2.5mm_P5.00mm, F.Cu at (401.4, 179.7)
- added C36: 100nF, Capacitor_THT:C_Disc_D5.0mm_W2.5mm_P5.00mm, F.Cu at (401.4, 183.8)
- added C37: 100nF, Capacitor_THT:C_Disc_D5.0mm_W2.5mm_P5.00mm, F.Cu at (393.0, 333.4)
- added D2: 1N4148, Diode_THT:D_DO-35_SOD27_P7.62mm_Horizontal, F.Cu at (457.8, 210.7)
- added D3: 1N4148, Diode_THT:D_DO-35_SOD27_P7.62mm_Horizontal, F.Cu at (377.8, 333.4)
- added J4: Barrel_Jack, Connector_BarrelJack:BarrelJack_CUI_PJ-063AH_Horizontal, F.Cu at (24.8, 398.1)
- added Q8: IRLZ44N, Package_TO_SOT_THT:TO-220-3_Vertical, F.Cu at (162.6, 366.7)
- added R124: 10k, Resistor_THT:R_Axial_DIN0204_L3.6mm_D1.6mm_P2.54mm_Vertical, F.Cu at (74.9, 348.6)
- added R6: 100k, Resistor_THT:R_Axial_DIN0204_L3.6mm_D1.6mm_P2.54mm_Vertical, F.Cu at (162.6, 360.7)
- C12, C9: footprint Capacitor_THT:CP_Axial_L10.0mm_D4.5mm_P15.00mm_Horizontal -> Capacitor_THT:CP_Radial_D5.0mm_P2.00mm
- Q5, Q6: value BS170 -> IRLZ44N; footprint Package_TO_SOT_THT:TO-92_Inline -> Package_TO_SOT_THT:TO-220-3_Vertical
- R100, R101, R102, R103, R104, R105, R106, R107, R108, R109, R110, R111, R112, R113, R114, R115, R116, R117, R118, R119, R120, R121, R122, R123, R15, R16, R17, R18, R19, R20, R21, R22, R23, R24, R25, R26, R51, R52, R55, R56, R57, R58, R59, R60, R61, R62, R63, R64, R68, R69, R70, R71, R72, R73, R74, R75, R76, R77, R78, R79, R80, R81, R82, R83, R84, R85, R86, R87, R88, R89, R90, R91, R92, R93, R94, R95, R96, R97, R98, R99: value 2.2k -> 1k
- SW2, SW3: footprint Button_Switch_THT:KSA_Tactile_SPST -> Button_Switch_THT:SW_PUSH_6mm_H4.3mm
- moved C7 448.9 mm to (426.1, 257.3)
- moved D48 448.8 mm to (359.1, 388.0), turned to 90 degrees
- moved D47 448.7 mm to (359.1, 382.9), turned to 90 degrees
- moved C1 441.9 mm to (432.5, 186.0)
- moved C2 441.9 mm to (432.5, 192.5)
- moved C3 441.9 mm to (432.5, 199.1)
- moved C4 441.9 mm to (432.5, 205.6)
- moved D56 438.2 mm to (338.8, 388.0), turned to 90 degrees
- moved D55 438.1 mm to (338.8, 382.9), turned to 90 degrees
- moved D50 438.1 mm to (354.0, 388.0), turned to 90 degrees
- moved D49 437.8 mm to (354.0, 382.9), turned to 90 degrees
- moved D14 433.5 mm to (304.8, 388.0), turned to 90 degrees
- moved D9 432.4 mm to (304.8, 382.9), turned to 90 degrees
- moved D52 427.8 mm to (349.0, 388.0), turned to 90 degrees
- moved D58 427.6 mm to (333.7, 388.0), turned to 90 degrees
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Connections:
- J3 pad 1: GND -> unconnected-(J3-Pin_1-Pad1)
- J3 pad 10: /D3 -> Net-(J3-Pin_10)
- J3 pad 4: /RS -> Net-(J3-Pin_4)
- J3 pad 5: /EN -> Net-(J3-Pin_5)
- J3 pad 6: /R/W -> Net-(J3-Pin_6)
- J3 pad 7: /D0 -> Net-(J3-Pin_7)
- J3 pad 8: /D1 -> Net-(J3-Pin_8)
- J3 pad 9: /D2 -> Net-(J3-Pin_9)
- Q5 pad 1: GND -> Net-(Q5-G)
- Q5 pad 2: Net-(Q5-G) -> Net-(Q5-D)
- Q6 pad 1: GND -> Net-(Q6-G)
- Q6 pad 2: Net-(Q6-G) -> Net-(Q5-D)
- R17 pad 1: Net-(R17-Pad1) -> Net-(Q2-D)
- R19 pad 1: Net-(U7-PA0) -> Net-(U7-CB2)
- R20 pad 1: Net-(U7-PA1) -> Net-(U7-CB1)
- R21 pad 1: Net-(U7-PA2) -> Net-(J3-Pin_10)
- R22 pad 1: Net-(U7-PA3) -> Net-(J3-Pin_9)
- R23 pad 1: Net-(U7-PA4) -> Net-(J3-Pin_8)
- R24 pad 1: Net-(U7-PA5) -> Net-(J3-Pin_7)
- R25 pad 1: Net-(U7-PA6) -> Net-(J3-Pin_6)
- R26 pad 1: Net-(U7-PA7) -> Net-(J3-Pin_5)
- R51 pad 1: Net-(U7-CB2) -> Net-(U7-PA0)
- R52 pad 1: Net-(U7-CB1) -> Net-(U7-PA1)
- R55 pad 1: Net-(U7-CA1) -> Net-(J3-Pin_4)
- R56 pad 1: Net-(U7-CA2) -> Net-(U7-PB0)
- R57 pad 1: Net-(U7-PB7) -> Net-(U7-PA2)
- R58 pad 1: /D3 -> Net-(U7-PA3)
- R59 pad 1: /RS -> Net-(U7-CA2)
- R60 pad 1: /EN -> Net-(U7-CA1)
- R61 pad 1: /R/W -> Net-(U7-PA7)
- R62 pad 1: /D0 -> Net-(U7-PA6)
- R63 pad 1: /D1 -> Net-(U7-PA5)
- R64 pad 1: /D2 -> Net-(U7-PA4)
- R68 pad 1: Net-(R17-Pad1) -> Net-(Q2-D)
- R70 pad 1: Net-(R17-Pad1) -> Net-(Q2-D)
- R71 pad 1: Net-(R17-Pad1) -> Net-(Q2-D)
- R73 pad 1: Net-(R17-Pad1) -> Net-(Q2-D)
- R75 pad 1: Net-(R17-Pad1) -> Net-(Q2-D)
- U1 pad 38: unconnected-(U1-~{SO}-Pad38) -> Net-(U1-~{SO})
- U12 pad 1: /A0 -> /D6
- U12 pad 10: Net-(D19-K) -> Net-(D14-A)
- U12 pad 11: /A4 -> /A1
- U12 pad 12: Net-(D21-K) -> Net-(D61-K)
- U12 pad 13: /A5 -> /D7
- U12 pad 2: Net-(D1-K) -> Net-(D59-K)
- U12 pad 3: /A2 -> /A0
- U12 pad 4: Net-(D15-K) -> Net-(D1-K)
- U12 pad 5: /A1 -> /A2
- U12 pad 6: Net-(D14-A) -> Net-(D15-K)
- U14 pad 11: unconnected-(U14-Pad11) -> GND
- U14 pad 13: unconnected-(U14-Pad13) -> GND
- U14 pad 5: unconnected-(U14-Pad5) -> GND
- U14 pad 9: unconnected-(U14-Pad9) -> GND
- U15 pad 1: unconnected-(U15-~{CKB}-Pad1) -> Net-(U15-Q0)
- U16 pad 1: /A6 -> /A4
- U16 pad 10: Net-(D33-K) -> Net-(D25-K)
- U16 pad 11: /A10 -> /A7
- U16 pad 12: Net-(D35-K) -> Net-(D21-K)
- U16 pad 13: /A11 -> /A5
- U16 pad 2: Net-(D23-K) -> Net-(D19-K)
- U16 pad 3: /A8 -> /A6
- U16 pad 4: Net-(D28-K) -> Net-(D23-K)
- U16 pad 5: /A7 -> /A8
- U16 pad 6: Net-(D25-K) -> Net-(D28-K)
- U17 pad 1: /A12 -> /A10
- U17 pad 10: Net-(D47-K) -> Net-(D41-K)
- U17 pad 11: /D0 -> /A13
- U17 pad 12: Net-(D49-K) -> Net-(D35-K)
- U17 pad 13: /D1 -> /A11
- U17 pad 2: Net-(D37-K) -> Net-(D33-K)
- U17 pad 3: /A15 -> /A12
- U17 pad 4: Net-(D43-K) -> Net-(D37-K)
- U17 pad 5: /A13 -> /A14
- U17 pad 6: Net-(D41-K) -> Net-(D43-K)
- U17 pad 9: /A9 -> /A15
- U18 pad 1: /D2 -> /D0
- U18 pad 10: Net-(D59-K) -> Net-(D53-K)
- U18 pad 11: /D6 -> /D3
- U18 pad 12: Net-(D61-K) -> Net-(D49-K)
- U18 pad 13: /D7 -> /D1
- U18 pad 2: Net-(D51-K) -> Net-(D47-K)
- U18 pad 3: /D4 -> /D2
- U18 pad 4: Net-(D55-K) -> Net-(D51-K)
- U18 pad 5: /D3 -> /D4
- U18 pad 6: Net-(D53-K) -> Net-(D55-K)
- U4 pad 1: (no net) -> GND
- U4 pad 2: (no net) -> GND
- U4 pad 3: (no net) -> unconnected-(U4-Pad3)
- U4 pad 4: Net-(U5-Qa) -> GND
- U4 pad 5: Net-(U5-Qa) -> GND
- U4 pad 6: phi0 -> unconnected-(U4-Pad6)
- U5 pad 7: Net-(U5-Qa) -> phi0
- U7 pad 10: /RS -> Net-(U7-PB0)
- U7 pad 11: /EN -> Net-(J3-Pin_4)
- U7 pad 12: /R/W -> Net-(J3-Pin_5)
- U7 pad 13: /D0 -> Net-(J3-Pin_6)
- U7 pad 14: /D1 -> Net-(J3-Pin_7)
- U7 pad 15: /D2 -> Net-(J3-Pin_8)
- U7 pad 16: /D3 -> Net-(J3-Pin_9)
- U7 pad 17: Net-(U7-PB7) -> Net-(J3-Pin_10)
Routing:
- net GND: track 874.8 -> 2525.5 mm, vias 1 -> 24
- net +5V: track 717.8 -> 2197.7 mm, vias 1 -> 22
- net /A0: track 639.0 -> 1000.5 mm, vias 1 -> 7
- net /A1: track 638.4 -> 996.2 mm, vias 1 -> 7
- net /A2: track 641.6 -> 980.4 mm, vias 1 -> 7
- net /A3: track 641.6 -> 978.1 mm, vias 1 -> 7
- net /D3: track 634.8 -> 960.8 mm, vias 1 -> 7
- net /D1: track 633.6 -> 949.1 mm, vias 1 -> 7
- net /D5: track 634.7 -> 948.1 mm, vias 1 -> 7
- net /D4: track 635.0 -> 946.9 mm, vias 1 -> 7
- net /D2: track 633.9 -> 944.7 mm, vias 1 -> 7
- net /D0: track 635.9 -> 938.9 mm, vias 1 -> 7
- net /D6: track 637.5 -> 939.6 mm, vias 1 -> 7
- net /D7: track 642.3 -> 943.4 mm, vias 1 -> 7
- net ROM CE: track 535.9 -> 240.7 mm, vias 0 -> 3
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- added copper zone on B.Cu, net (none)
- added copper zone on F.Cu, net (none)
- added copper zone on B.Cu, net GND
- added copper zone on F.Cu, net GND
Other:
- board text added: "1"
- board text added: "1MHz CLOCK"
- board text added: "5V / 1A"
- board text added: "A0"
- board text added: "A15"
- board text added: "ADDRESS BUS"
- board text added: "CLOCK SWITCH"
- board text added: "CONTROL SIGNALS"
- board text added: "CSb PERIPHERAL"
- board text added: "D0"
- board text added: "D7"
- board text added: "DATA BUS"
- board text added: "RESET"
- board text added: "STEP"
- board text added: "STEP CLOCK"
- board text added: "SWITCH"
- board text added: "TODO: RP2040 board here"
- board text added: "VARIABLE CLOCK"

Commit message: finish 1st placing
Parts:
- J2: footprint Connector_Dsub:DSUB-9_Socket_EdgeMount_P2.77mm -> Connector_Dsub:DSUB-9_Pins_Horizontal_P2.77x2.84mm_EdgePinOffset4.94mm_Housed_MountingHolesOffset4.94mm
- RV1: footprint Potentiometer_THT:Potentiometer_ACP_CA6-H2,5_Horizontal -> Potentiometer_THT:Potentiometer_Alpha_RD901F-40-00D_Single_Vertical
- moved C25 373.2 mm to (55.9, 331.5)
- moved C32 339.6 mm to (102.9, 329.6)
- moved C33 319.8 mm to (123.3, 329.6)
- moved C34 299.2 mm to (144.8, 329.6)
- moved C35 80.5 mm to (411.5, 259.6), turned to 90 degrees
- moved C36 76.9 mm to (400.7, 260.7), turned to 180 degrees
- moved C1 66.8 mm to (377.8, 224.5)
- moved C2 64.9 mm to (425.4, 257.0)
- moved D2 57.7 mm to (403.2, 229.6)
- moved C4 55.8 mm to (421.0, 260.2), turned to 180 degrees
- moved C3 50.8 mm to (425.4, 249.4)
- moved U10 30.6 mm to (422.3, 257.0), turned to 180 degrees
- moved Y2 21.4 mm to (378.5, 240.9)
- moved J2 14.5 mm to (436.0, 248.3)
- moved U6 13.6 mm to (385.4, 224.5)
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Connections:
- R21 pad 1: Net-(J3-Pin_10) -> Net-(J3-Pin_4)
- R22 pad 1: Net-(J3-Pin_9) -> Net-(J3-Pin_5)
- R23 pad 1: Net-(J3-Pin_8) -> Net-(J3-Pin_6)
- R25 pad 1: Net-(J3-Pin_6) -> Net-(J3-Pin_8)
- R26 pad 1: Net-(J3-Pin_5) -> Net-(J3-Pin_9)
- R55 pad 1: Net-(J3-Pin_4) -> Net-(J3-Pin_10)
- U7 pad 11: Net-(J3-Pin_4) -> Net-(J3-Pin_10)
- U7 pad 12: Net-(J3-Pin_5) -> Net-(J3-Pin_9)
- U7 pad 13: Net-(J3-Pin_6) -> Net-(J3-Pin_8)
- U7 pad 15: Net-(J3-Pin_8) -> Net-(J3-Pin_6)
- U7 pad 16: Net-(J3-Pin_9) -> Net-(J3-Pin_5)
- U7 pad 17: Net-(J3-Pin_10) -> Net-(J3-Pin_4)
Routing:
- net /A15: track 823.9 -> 513.4 mm, vias 6 -> 5
- net /A12: track 821.9 -> 512.1 mm
- net BE: track 674.1 -> 364.3 mm
- net /A14: track 865.0 -> 555.9 mm
- net /A11: track 905.1 -> 597.2 mm
- net /A6: track 874.4 -> 586.8 mm
- net /A4: track 891.6 -> 605.2 mm
- net /A5: track 889.4 -> 603.6 mm
- net /A8: track 889.7 -> 604.0 mm
- net /A7: track 870.9 -> 585.2 mm, vias 7 -> 6
- net RAM CS: track 535.2 -> 259.7 mm
- net /A9: track 902.6 -> 627.8 mm
- net /A2: track 980.4 -> 782.2 mm
- net +5V: track 2197.7 -> 2001.5 mm, vias 22 -> 25
- net /A3: track 978.1 -> 781.8 mm
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- removed copper zone on B.Cu, net GND
Other:
- board outline added: 502.9 x 199.4 mm
- board text added: "CHANGE CLOCK"
- board text added: "FIXME: mouting holes 60x98"
- board text added: "TODO: - edge - f.mask fill-in - backplane gnd - fix segment layout"
- board text removed: "CLOCK SWITCH"
- board text removed: "STEP"
- board text removed: "SWITCH"
- board text removed: "TODO: RP2040 board here"

Commit message: update todo
Other:
- board text added: "TODO: - edge - f.mask fill-in - backplane gnd - fix segment layout - find proper components and fix footprints (potmeter, diodes, db9, barrel jack, ..) - create rp2040 board - measure mounting holes for display - put mounting holes"
- board text removed: "TODO: - edge - f.mask fill-in - backplane gnd - fix segment layout"
Changed lines of the file:
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@@
 		)
 	)
-	(gr_text "TODO:\n- edge\n- f.mask fill-in\n- backplane gnd\n- fix segment layout"
-		(at 483.235 247.015 0)
+	(gr_text "TODO:\n- edge\n- f.mask fill-in\n- backplane gnd\n- fix segment layout\n- find proper components and fix footprints (potmeter, diodes, db9, barrel jack, ..)\n- create rp2040 board\n- measure mounting holes for display\n- put mounting holes"
+		(at 266.5 225 0)
 		(layer "User.4")
 		(effects

Commit message: fix DRC errors
Routing:
- net GND: track 2487.0 -> 2473.3 mm
- net Net-(U21-D3): track 14.9 -> 21.4 mm
- net Net-(Q7-B): track 15.8 -> 21.3 mm
- net Net-(Q5-S): track 158.2 -> 160.2 mm
- net Net-(U22-E): track 27.0 -> 25.5 mm
- net Net-(U25-E): track 26.9 -> 25.4 mm
- net Net-(U28-G): track 20.8 -> 22.3 mm
- net Net-(U22-G): track 20.9 -> 22.2 mm, vias 0 -> 1
- net Net-(C14-Pad1): track 50.9 -> 52.2 mm
- net Net-(U11-Q): track 69.3 -> 70.5 mm
- net Net-(U25-F): track 23.3 -> 24.5 mm, vias 0 -> 1
- net Net-(U28-E): track 26.9 -> 26.0 mm
- net Net-(U27-D5): track 10.4 -> 11.0 mm
- net /A0: track 882.4 -> 881.8 mm
- net Net-(U28-C): track 20.8 -> 21.4 mm
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
Commit message: fix ERC and DRC problems
Connections:
- J3 pad 1: unconnected-(J3-Pin_1-Pad1) -> GND
Routing:
- net GND: track 2473.3 -> 2487.9 mm

Commit message: ground plane + mounting holes
Parts:
- added REF**: MountingHole_3.2mm_M3, MountingHole:MountingHole_3.2mm_M3, F.Cu at (510.5, 213.4)
- added REF**: MountingHole_3.2mm_M3, MountingHole:MountingHole_3.2mm_M3, F.Cu at (510.5, 403.9)
- added REF**: MountingHole_3.2mm_M3, MountingHole:MountingHole_3.2mm_M3, F.Cu at (16.5, 403.2)
- added REF**: MountingHole_3.2mm_M3, MountingHole:MountingHole_3.2mm_M3, F.Cu at (16.5, 213.4)
Routing:
- net +5V: track 2001.1 -> 2178.9 mm
- net GND: track 2487.9 -> 2662.5 mm, vias 26 -> 36
- net SW_BUS_DEC: track 190.9 -> 189.4 mm, vias 2 -> 1
- added copper zone on B.Cu, net GND
- removed copper zone on B.Cu, net (none)
- removed copper zone on F.Cu, net (none)
Other:
- board text added: "TODO: - find proper components and fix footprints (potmeter, diodes, db9, barrel jack, ..) - create rp2040 board - measure mounting holes for display - put mounting holes on whole board"
- board text removed: "TODO: - edge - f.mask fill-in - backplane gnd - fix segment layout - find proper components and fix footprints (potmeter, diodes, db9, barrel jack, ..) - create rp2040 board - measure mounting holes for display - put mounting holes"

Commit message: finish board
Parts:
- removed C15: 1000uF, Capacitor_THT:CP_Axial_L20.0mm_D10.0mm_P26.00mm_Horizontal
- moved C13 11.4 mm to (84.3, 251.5)
- moved SW3 11.4 mm to (85.8, 247.7)
- moved REF** 9.52 mm to (26.0, 403.2)
- moved J4 9.00 mm to (33.8, 388.6)
- moved C10 8.26 mm to (95.9, 215.3)
- moved C30 8.26 mm to (95.9, 229.2)
- moved RV1 8.26 mm to (79.4, 227.0)
- moved C11 8.26 mm to (46.4, 217.2)
- moved C12 8.26 mm to (50.8, 217.2)
- moved C18 8.26 mm to (67.9, 261.6)
- moved C31 8.26 mm to (52.1, 261.6)
- moved R10 8.26 mm to (51.4, 224.8)
- moved R13 8.26 mm to (70.5, 261.6)
- moved SW2 8.26 mm to (71.3, 221.7)
- moved U13 8.26 mm to (61.6, 229.9)
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Routing:
- net GND: track 2662.5 -> 0.00 mm, vias 36 -> 8
- net +5V: track 2178.9 -> 2144.2 mm
- net Net-(U10-T1OUT): track 27.6 -> 39.7 mm
- net Net-(U10-R1IN): track 27.6 -> 38.1 mm
- net RESb: track 550.2 -> 540.9 mm
- net IRQb: track 603.7 -> 598.0 mm
- net /D2: track 856.4 -> 850.7 mm
- net /D0: track 841.2 -> 835.5 mm
- net /A13: track 698.2 -> 692.5 mm
- net /A10: track 813.4 -> 807.7 mm
- net phi0: track 650.9 -> 645.2 mm
- net /D3: track 875.4 -> 869.6 mm
- net /A2: track 782.2 -> 776.5 mm
- net /A0: track 881.8 -> 876.1 mm
- net /A3: track 781.8 -> 776.1 mm
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Other:
- board size 502.9 x 199.4 mm -> 488.9 x 198.8 mm
- board text added: "ADDRESS DECODER"
- board text added: "LED CONTROL"
- board text added: "TODO: - find proper components and fix footprints (potmeter, diodes, db9, barrel jack, ..) - create rp2040 board - measure mounting holes for display"
- board text removed: "GND"
- board text removed: "TODO: - find proper components and fix footprints (potmeter, diodes, db9, barrel jack, ..) - create rp2040 board - measure mounting holes for display - put mounting holes on whole board"
