File: wallputer-modular/power-card/power-card.kicad_pcb (KiCad board)
At the start: 2 copper layers, 1 part

Commit message: footprints
Parts:
- added C1: 100nF, Capacitor_THT:C_Disc_D5.0mm_W2.5mm_P5.00mm, F.Cu at (-62.3, 97.1)
- added C19: 100nF, Capacitor_THT:C_Disc_D5.0mm_W2.5mm_P5.00mm, F.Cu at (-27.0, 79.1)
- added C2: 0.01uF, Capacitor_THT:C_Disc_D5.0mm_W2.5mm_P5.00mm, F.Cu at (-62.3, 101.1)
- added C20: 100nF, Capacitor_THT:C_Disc_D5.0mm_W2.5mm_P5.00mm, F.Cu at (-27.0, 83.1)
- added C21: 100nF, Capacitor_THT:C_Disc_D5.0mm_W2.5mm_P5.00mm, F.Cu at (-27.0, 87.2)
- added C22: 100nF, Capacitor_THT:C_Disc_D5.0mm_W2.5mm_P5.00mm, F.Cu at (-27.0, 91.2)
- added C3: 4.7nF, Capacitor_THT:C_Disc_D5.0mm_W2.5mm_P5.00mm, F.Cu at (-62.3, 105.2)
- added C4: 100nF, Capacitor_THT:C_Disc_D5.0mm_W2.5mm_P5.00mm, F.Cu at (-27.0, 71.0)
- added C5: 100nF, Capacitor_THT:C_Disc_D5.0mm_W2.5mm_P5.00mm, F.Cu at (-27.0, 75.0)
- added C6: 0.1uF, Capacitor_THT:C_Disc_D5.0mm_W2.5mm_P5.00mm, F.Cu at (-78.2, 92.1)
- added C7: 2000uF, Capacitor_THT:CP_Radial_D18.0mm_P7.50mm, F.Cu at (26.7, 188.5)
- added D1: Green LED, LED_THT:LED_D3.0mm, F.Cu at (-84.0, 33.9)
- added D10: Green LED, LED_THT:LED_D3.0mm, F.Cu at (-84.0, 72.2)
- added D11: Red LED, LED_THT:LED_D3.0mm, F.Cu at (-84.0, 77.7)
- added D12: Green LED, LED_THT:LED_D3.0mm, F.Cu at (-84.0, 83.1)
- added D13: Red LED, LED_THT:LED_D3.0mm, F.Cu at (-78.1, 33.9)
- added D14: Red LED, LED_THT:LED_D3.0mm, F.Cu at (-78.1, 39.4)
- added D15: Green LED, LED_THT:LED_D3.0mm, F.Cu at (-78.1, 44.8)
- added D16: Red LED, LED_THT:LED_D3.0mm, F.Cu at (-78.1, 50.3)
- added D17: Green LED, LED_THT:LED_D3.0mm, F.Cu at (-78.1, 55.8)
- added D18: Red LED, LED_THT:LED_D3.0mm, F.Cu at (-78.1, 61.2)
- added D19: Green LED, LED_THT:LED_D3.0mm, F.Cu at (-78.1, 66.7)
- added D2: 1n4148, Diode_THT:D_DO-35_SOD27_P7.62mm_Horizontal, F.Cu at (-65.4, 110.7)
- added D20: Red LED, LED_THT:LED_D3.0mm, F.Cu at (-78.1, 72.2)
- added D21: Green LED, LED_THT:LED_D3.0mm, F.Cu at (-78.1, 77.7)
- added D22: Red LED, LED_THT:LED_D3.0mm, F.Cu at (-78.1, 83.1)
- added D23: Green LED, LED_THT:LED_D3.0mm, F.Cu at (-72.2, 33.9)
- added D24: Red LED, LED_THT:LED_D3.0mm, F.Cu at (-72.2, 39.4)
- added D25: Green LED, LED_THT:LED_D3.0mm, F.Cu at (-72.2, 44.8)
- added D26: Red LED, LED_THT:LED_D3.0mm, F.Cu at (-72.2, 50.3)
- added D27: Green LED, LED_THT:LED_D3.0mm, F.Cu at (-72.2, 55.8)
- added D28: Green LED, LED_THT:LED_D3.0mm, F.Cu at (-72.2, 61.2)
- added D29: Red LED, LED_THT:LED_D3.0mm, F.Cu at (-72.2, 66.7)
- added D3: 1n4148, Diode_THT:D_DO-35_SOD27_P7.62mm_Horizontal, F.Cu at (-65.4, 114.3)
- added D30: Red LED, LED_THT:LED_D3.0mm, F.Cu at (-72.2, 72.2)
- added D31: Green LED, LED_THT:LED_D3.0mm, F.Cu at (-72.2, 77.7)
- added D32: Red LED, LED_THT:LED_D3.0mm, F.Cu at (-72.2, 83.1)
- added D33: Green LED, LED_THT:LED_D3.0mm, F.Cu at (-66.4, 33.9)
- added D34: Red LED, LED_THT:LED_D3.0mm, F.Cu at (-66.4, 39.4)
- added D35: Green LED, LED_THT:LED_D3.0mm, F.Cu at (-66.4, 44.8)
- added D36: Red LED, LED_THT:LED_D3.0mm, F.Cu at (-66.4, 50.3)
- added D37: Green LED, LED_THT:LED_D3.0mm, F.Cu at (-66.4, 55.8)
- added D38: Green LED, LED_THT:LED_D3.0mm, F.Cu at (-66.4, 61.2)
- added D39: Red LED, LED_THT:LED_D3.0mm, F.Cu at (-66.4, 66.7)
- added D4: Green LED, LED_THT:LED_D3.0mm, F.Cu at (-84.0, 39.4)
- added D40: Red LED, LED_THT:LED_D3.0mm, F.Cu at (-66.4, 72.2)
- added D41: Green LED, LED_THT:LED_D3.0mm, F.Cu at (-66.4, 77.7)
- added D42: Red LED, LED_THT:LED_D3.0mm, F.Cu at (-66.4, 83.1)
- added D43: Green LED, LED_THT:LED_D3.0mm, F.Cu at (-60.5, 33.9)
- added D44: Red LED, LED_THT:LED_D3.0mm, F.Cu at (-60.5, 39.4)
- added D45: Green LED, LED_THT:LED_D3.0mm, F.Cu at (-60.5, 44.8)
- added D46: Red LED, LED_THT:LED_D3.0mm, F.Cu at (-60.5, 50.3)
- added D47: Green LED, LED_THT:LED_D3.0mm, F.Cu at (-60.5, 55.8)
- added D48: Red LED, LED_THT:LED_D3.0mm, F.Cu at (-60.5, 61.2)
- added D49: Green LED, LED_THT:LED_D3.0mm, F.Cu at (-60.5, 66.7)
- added D5: Red LED, LED_THT:LED_D3.0mm, F.Cu at (-84.0, 44.8)
- added D50: Red LED, LED_THT:LED_D3.0mm, F.Cu at (-60.5, 72.2)
- added D51: Green LED, LED_THT:LED_D3.0mm, F.Cu at (-60.5, 77.7)
- added D52: Red LED, LED_THT:LED_D3.0mm, F.Cu at (-60.5, 83.1)
- added D53: Green LED, LED_THT:LED_D3.0mm, F.Cu at (-54.6, 33.9)
- added D54: Red LED, LED_THT:LED_D3.0mm, F.Cu at (-54.6, 39.4)
- added D55: Green LED, LED_THT:LED_D3.0mm, F.Cu at (-54.6, 44.8)
- added D56: Red LED, LED_THT:LED_D3.0mm, F.Cu at (-54.6, 50.3)
- added D57: Green LED, LED_THT:LED_D3.0mm, F.Cu at (-54.6, 55.8)
- added D58: Red LED, LED_THT:LED_D3.0mm, F.Cu at (-54.6, 61.2)
- added D59: Green LED, LED_THT:LED_D3.0mm, F.Cu at (-54.6, 66.7)
- added D6: Red LED, LED_THT:LED_D3.0mm, F.Cu at (-84.0, 50.3)
- added D60: Red LED, LED_THT:LED_D3.0mm, F.Cu at (-54.6, 72.2)
- added D61: Green LED, LED_THT:LED_D3.0mm, F.Cu at (-54.6, 77.7)
- added D62: Red LED, LED_THT:LED_D3.0mm, F.Cu at (-54.6, 83.1)
- added D63: Green LED, LED_THT:LED_D3.0mm, F.Cu at (-48.7, 33.9)
- added D64: Red LED, LED_THT:LED_D3.0mm, F.Cu at (-48.7, 39.4)
- added D65: Green LED, LED_THT:LED_D3.0mm, F.Cu at (-48.7, 44.8)
- added D66: Red LED, LED_THT:LED_D3.0mm, F.Cu at (-48.7, 50.3)
- added D67: Green LED, LED_THT:LED_D3.0mm, F.Cu at (-48.7, 55.8)
- added D68: Red LED, LED_THT:LED_D3.0mm, F.Cu at (-48.7, 61.2)
- added D69: Green LED, LED_THT:LED_D3.0mm, F.Cu at (-48.7, 66.7)
- added D7: Green LED, LED_THT:LED_D3.0mm, F.Cu at (-84.0, 55.8)
- added D70: Red LED, LED_THT:LED_D3.0mm, F.Cu at (-48.7, 72.2)
- added D71: Green LED, LED_THT:LED_D3.0mm, F.Cu at (-48.7, 77.7)
- added D72: Red LED, LED_THT:LED_D3.0mm, F.Cu at (-48.7, 83.1)
- added D8: Red LED, LED_THT:LED_D3.0mm, F.Cu at (-84.0, 61.2)
- added D9: Green LED, LED_THT:LED_D3.0mm, F.Cu at (-84.0, 66.7)
- added J2: Power, Connector_USB:USB_C_Receptacle_HRO_TYPE-C-31-M-12, F.Cu at (20.7, 164.6)
- added Q1: FQP27P06, Package_TO_SOT_THT:TO-220-3_Vertical, F.Cu at (-12.2, 15.6)
- added Q2: IRLZ44N, Package_TO_SOT_THT:TO-220-3_Vertical, F.Cu at (-12.2, 21.6)
- added R1: 5.1k, Resistor_THT:R_Axial_DIN0204_L3.6mm_D1.6mm_P2.54mm_Vertical, F.Cu at (-83.8, 91.6)
- added R10: 1k, Resistor_THT:R_Axial_DIN0204_L3.6mm_D1.6mm_P2.54mm_Vertical, F.Cu at (-27.0, 48.5)
- added R100: 1k, Resistor_THT:R_Axial_DIN0204_L3.6mm_D1.6mm_P2.54mm_Vertical, F.Cu at (-4.63, 64.2)
- added R101: 1k, Resistor_THT:R_Axial_DIN0204_L3.6mm_D1.6mm_P2.54mm_Vertical, F.Cu at (-4.63, 67.4)
- added R102: 1k, Resistor_THT:R_Axial_DIN0204_L3.6mm_D1.6mm_P2.54mm_Vertical, F.Cu at (0.96, 32.7)
- added R103: 1k, Resistor_THT:R_Axial_DIN0204_L3.6mm_D1.6mm_P2.54mm_Vertical, F.Cu at (0.96, 35.9)
- added R104: 1k, Resistor_THT:R_Axial_DIN0204_L3.6mm_D1.6mm_P2.54mm_Vertical, F.Cu at (0.96, 39.0)
- added R105: 1k, Resistor_THT:R_Axial_DIN0204_L3.6mm_D1.6mm_P2.54mm_Vertical, F.Cu at (0.96, 42.2)
- added R106: 1k, Resistor_THT:R_Axial_DIN0204_L3.6mm_D1.6mm_P2.54mm_Vertical, F.Cu at (0.96, 45.3)
- added R107: 1k, Resistor_THT:R_Axial_DIN0204_L3.6mm_D1.6mm_P2.54mm_Vertical, F.Cu at (0.96, 48.5)
- added R108: 1k, Resistor_THT:R_Axial_DIN0204_L3.6mm_D1.6mm_P2.54mm_Vertical, F.Cu at (0.96, 51.6)
- added R109: 1k, Resistor_THT:R_Axial_DIN0204_L3.6mm_D1.6mm_P2.54mm_Vertical, F.Cu at (0.96, 54.8)
- added R11: 1k, Resistor_THT:R_Axial_DIN0204_L3.6mm_D1.6mm_P2.54mm_Vertical, F.Cu at (-27.0, 51.6)
- added R110: 1k, Resistor_THT:R_Axial_DIN0204_L3.6mm_D1.6mm_P2.54mm_Vertical, F.Cu at (0.96, 57.9)
- added R111: 1k, Resistor_THT:R_Axial_DIN0204_L3.6mm_D1.6mm_P2.54mm_Vertical, F.Cu at (0.96, 61.1)
- added R12: 1k, Resistor_THT:R_Axial_DIN0204_L3.6mm_D1.6mm_P2.54mm_Vertical, F.Cu at (-27.0, 54.8)
- added R13: 1k, Resistor_THT:R_Axial_DIN0204_L3.6mm_D1.6mm_P2.54mm_Vertical, F.Cu at (-27.0, 57.9)
- added R14: 1k, Resistor_THT:R_Axial_DIN0204_L3.6mm_D1.6mm_P2.54mm_Vertical, F.Cu at (-27.0, 61.1)
- added R15: 1k, Resistor_THT:R_Axial_DIN0204_L3.6mm_D1.6mm_P2.54mm_Vertical, F.Cu at (-27.0, 64.2)
- added R16: 1k, Resistor_THT:R_Axial_DIN0204_L3.6mm_D1.6mm_P2.54mm_Vertical, F.Cu at (-27.0, 67.4)
- added R17: 1k, Resistor_THT:R_Axial_DIN0204_L3.6mm_D1.6mm_P2.54mm_Vertical, F.Cu at (-21.4, 32.7)
- added R18: 1k, Resistor_THT:R_Axial_DIN0204_L3.6mm_D1.6mm_P2.54mm_Vertical, F.Cu at (-21.4, 35.9)
- added R19: 1k, Resistor_THT:R_Axial_DIN0204_L3.6mm_D1.6mm_P2.54mm_Vertical, F.Cu at (-21.4, 39.0)
- added R2: 5.1k, Resistor_THT:R_Axial_DIN0204_L3.6mm_D1.6mm_P2.54mm_Vertical, F.Cu at (-83.8, 94.8)
- added R20: 1k, Resistor_THT:R_Axial_DIN0204_L3.6mm_D1.6mm_P2.54mm_Vertical, F.Cu at (-21.4, 42.2)
- added R21: 1k, Resistor_THT:R_Axial_DIN0204_L3.6mm_D1.6mm_P2.54mm_Vertical, F.Cu at (-21.4, 45.3)
- added R22: 1k, Resistor_THT:R_Axial_DIN0204_L3.6mm_D1.6mm_P2.54mm_Vertical, F.Cu at (-21.4, 48.5)
- added R23: 1k, Resistor_THT:R_Axial_DIN0204_L3.6mm_D1.6mm_P2.54mm_Vertical, F.Cu at (-21.4, 51.6)
- added R24: 1k, Resistor_THT:R_Axial_DIN0204_L3.6mm_D1.6mm_P2.54mm_Vertical, F.Cu at (-21.4, 54.8)
- added R25: 1k, Resistor_THT:R_Axial_DIN0204_L3.6mm_D1.6mm_P2.54mm_Vertical, F.Cu at (-21.4, 57.9)
- added R26: 1k, Resistor_THT:R_Axial_DIN0204_L3.6mm_D1.6mm_P2.54mm_Vertical, F.Cu at (-21.4, 61.1)
- added R27: 1k, Resistor_THT:R_Axial_DIN0204_L3.6mm_D1.6mm_P2.54mm_Vertical, F.Cu at (-21.4, 64.2)
- added R28: 1k, Resistor_THT:R_Axial_DIN0204_L3.6mm_D1.6mm_P2.54mm_Vertical, F.Cu at (-21.4, 67.4)
- added R29: 1k, Resistor_THT:R_Axial_DIN0204_L3.6mm_D1.6mm_P2.54mm_Vertical, F.Cu at (-15.8, 32.7)
- added R3: 1k, Resistor_THT:R_Axial_DIN0204_L3.6mm_D1.6mm_P2.54mm_Vertical, F.Cu at (-83.8, 97.9)
- added R30: 1k, Resistor_THT:R_Axial_DIN0204_L3.6mm_D1.6mm_P2.54mm_Vertical, F.Cu at (-15.8, 35.9)
- added R31: 10k, Resistor_THT:R_Axial_DIN0204_L3.6mm_D1.6mm_P2.54mm_Vertical, F.Cu at (-83.8, 104.2)
- added R32: 220, Resistor_THT:R_Axial_DIN0204_L3.6mm_D1.6mm_P2.54mm_Vertical, F.Cu at (-83.8, 107.4)
- added R33: 10k, Resistor_THT:R_Axial_DIN0204_L3.6mm_D1.6mm_P2.54mm_Vertical, F.Cu at (-83.8, 110.5)
- added R34: 100k, Resistor_THT:R_Axial_DIN0204_L3.6mm_D1.6mm_P2.54mm_Vertical, F.Cu at (-83.8, 113.7)
- added R4: 220, Resistor_THT:R_Axial_DIN0204_L3.6mm_D1.6mm_P2.54mm_Vertical, F.Cu at (-83.8, 101.1)
- added R5: 1k, Resistor_THT:R_Axial_DIN0204_L3.6mm_D1.6mm_P2.54mm_Vertical, F.Cu at (-27.0, 32.7)
- added R6: 1k, Resistor_THT:R_Axial_DIN0204_L3.6mm_D1.6mm_P2.54mm_Vertical, F.Cu at (-27.0, 35.9)
- added R68: 1k, Resistor_THT:R_Axial_DIN0204_L3.6mm_D1.6mm_P2.54mm_Vertical, F.Cu at (-15.8, 39.0)
- added R69: 1k, Resistor_THT:R_Axial_DIN0204_L3.6mm_D1.6mm_P2.54mm_Vertical, F.Cu at (-15.8, 42.2)
- added R7: 1k, Resistor_THT:R_Axial_DIN0204_L3.6mm_D1.6mm_P2.54mm_Vertical, F.Cu at (-27.0, 39.0)
- added R70: 1k, Resistor_THT:R_Axial_DIN0204_L3.6mm_D1.6mm_P2.54mm_Vertical, F.Cu at (-15.8, 45.3)
- added R71: 1k, Resistor_THT:R_Axial_DIN0204_L3.6mm_D1.6mm_P2.54mm_Vertical, F.Cu at (-15.8, 48.5)
- added R72: 1k, Resistor_THT:R_Axial_DIN0204_L3.6mm_D1.6mm_P2.54mm_Vertical, F.Cu at (-15.8, 51.6)
- added R73: 1k, Resistor_THT:R_Axial_DIN0204_L3.6mm_D1.6mm_P2.54mm_Vertical, F.Cu at (-15.8, 54.8)
- added R74: 1k, Resistor_THT:R_Axial_DIN0204_L3.6mm_D1.6mm_P2.54mm_Vertical, F.Cu at (-15.8, 57.9)
- added R75: 1k, Resistor_THT:R_Axial_DIN0204_L3.6mm_D1.6mm_P2.54mm_Vertical, F.Cu at (-15.8, 61.1)
- added R76: 1k, Resistor_THT:R_Axial_DIN0204_L3.6mm_D1.6mm_P2.54mm_Vertical, F.Cu at (-15.8, 64.2)
- added R77: 1k, Resistor_THT:R_Axial_DIN0204_L3.6mm_D1.6mm_P2.54mm_Vertical, F.Cu at (-15.8, 67.4)
- added R78: 1k, Resistor_THT:R_Axial_DIN0204_L3.6mm_D1.6mm_P2.54mm_Vertical, F.Cu at (-10.2, 32.7)
- added R79: 1k, Resistor_THT:R_Axial_DIN0204_L3.6mm_D1.6mm_P2.54mm_Vertical, F.Cu at (-10.2, 35.9)
- added R8: 1k, Resistor_THT:R_Axial_DIN0204_L3.6mm_D1.6mm_P2.54mm_Vertical, F.Cu at (-27.0, 42.2)
- added R80: 1k, Resistor_THT:R_Axial_DIN0204_L3.6mm_D1.6mm_P2.54mm_Vertical, F.Cu at (-10.2, 39.0)
- added R81: 1k, Resistor_THT:R_Axial_DIN0204_L3.6mm_D1.6mm_P2.54mm_Vertical, F.Cu at (-10.2, 42.2)
- added R82: 1k, Resistor_THT:R_Axial_DIN0204_L3.6mm_D1.6mm_P2.54mm_Vertical, F.Cu at (-10.2, 45.3)
- added R83: 1k, Resistor_THT:R_Axial_DIN0204_L3.6mm_D1.6mm_P2.54mm_Vertical, F.Cu at (-10.2, 48.5)
- added R84: 1k, Resistor_THT:R_Axial_DIN0204_L3.6mm_D1.6mm_P2.54mm_Vertical, F.Cu at (-10.2, 51.6)
- added R85: 1k, Resistor_THT:R_Axial_DIN0204_L3.6mm_D1.6mm_P2.54mm_Vertical, F.Cu at (-10.2, 54.8)
- added R86: 1k, Resistor_THT:R_Axial_DIN0204_L3.6mm_D1.6mm_P2.54mm_Vertical, F.Cu at (-10.2, 57.9)
- added R87: 1k, Resistor_THT:R_Axial_DIN0204_L3.6mm_D1.6mm_P2.54mm_Vertical, F.Cu at (-10.2, 61.1)
- added R88: 1k, Resistor_THT:R_Axial_DIN0204_L3.6mm_D1.6mm_P2.54mm_Vertical, F.Cu at (-10.2, 64.2)
- added R89: 1k, Resistor_THT:R_Axial_DIN0204_L3.6mm_D1.6mm_P2.54mm_Vertical, F.Cu at (-10.2, 67.4)
- added R9: 1k, Resistor_THT:R_Axial_DIN0204_L3.6mm_D1.6mm_P2.54mm_Vertical, F.Cu at (-27.0, 45.3)
- added R90: 1k, Resistor_THT:R_Axial_DIN0204_L3.6mm_D1.6mm_P2.54mm_Vertical, F.Cu at (-4.63, 32.7)
- added R91: 1k, Resistor_THT:R_Axial_DIN0204_L3.6mm_D1.6mm_P2.54mm_Vertical, F.Cu at (-4.63, 35.9)
- added R92: 1k, Resistor_THT:R_Axial_DIN0204_L3.6mm_D1.6mm_P2.54mm_Vertical, F.Cu at (-4.63, 39.0)
- added R93: 1k, Resistor_THT:R_Axial_DIN0204_L3.6mm_D1.6mm_P2.54mm_Vertical, F.Cu at (-4.63, 42.2)
- added R94: 1k, Resistor_THT:R_Axial_DIN0204_L3.6mm_D1.6mm_P2.54mm_Vertical, F.Cu at (-4.63, 45.3)
- added R95: 1k, Resistor_THT:R_Axial_DIN0204_L3.6mm_D1.6mm_P2.54mm_Vertical, F.Cu at (-4.63, 48.5)
- added R96: 1k, Resistor_THT:R_Axial_DIN0204_L3.6mm_D1.6mm_P2.54mm_Vertical, F.Cu at (-4.63, 51.6)
- added R97: 1k, Resistor_THT:R_Axial_DIN0204_L3.6mm_D1.6mm_P2.54mm_Vertical, F.Cu at (-4.63, 54.8)
- added R98: 1k, Resistor_THT:R_Axial_DIN0204_L3.6mm_D1.6mm_P2.54mm_Vertical, F.Cu at (-4.63, 57.9)
- added R99: 1k, Resistor_THT:R_Axial_DIN0204_L3.6mm_D1.6mm_P2.54mm_Vertical, F.Cu at (-4.63, 61.1)
- added RV1: 50k, Potentiometer_THT:Potentiometer_Alpha_RD901F-40-00D_Single_Vertical, F.Cu at (47.1, 183.2)
- added SW1: reset, Button_Switch_THT:SW_PUSH_6mm_H4.3mm, F.Cu at (17.6, 147.9)
- added U1: NE555P, Package_DIP:DIP-8_W7.62mm, F.Cu at (67.9, 182.9)
- added U12: 74HC04, Package_DIP:DIP-14_W7.62mm_Socket, F.Cu at (-60.2, 13.8)
- added U16: 74HC04, Package_DIP:DIP-14_W7.62mm_Socket, F.Cu at (-48.5, 13.8)
- added U17: 74HC04, Package_DIP:DIP-14_W7.62mm_Socket, F.Cu at (-36.8, 13.8)
- added U18: 74HC04, Package_DIP:DIP-14_W7.62mm_Socket, F.Cu at (-25.1, 13.8)
- added U2: 74HC04, Package_DIP:DIP-14_W7.62mm_Socket, F.Cu at (-83.7, 13.8)
- added U3: 74HC04, Package_DIP:DIP-14_W7.62mm_Socket, F.Cu at (-71.9, 13.8)
- moved J1 241.0 mm to (-30.9, 33.4), turned to 0 degrees
Connections:
- J1 pad 1: unconnected-(J1-Vss-Pad1) -> GND
- J1 pad 10: unconnected-(J1-A5-Pad10) -> /A5
- J1 pad 11: unconnected-(J1-A6-Pad11) -> /A6
- J1 pad 12: unconnected-(J1-A7-Pad12) -> /A7
- J1 pad 13: unconnected-(J1-A8-Pad13) -> /A8
- J1 pad 14: unconnected-(J1-A9-Pad14) -> /A9
- J1 pad 15: unconnected-(J1-A10-Pad15) -> /A10
- J1 pad 16: unconnected-(J1-A11-Pad16) -> /A11
- J1 pad 17: unconnected-(J1-A12-Pad17) -> /A12
- J1 pad 18: unconnected-(J1-A13-Pad18) -> /A13
- J1 pad 19: unconnected-(J1-A14-Pad19) -> /A14
- J1 pad 2: unconnected-(J1-NC-Pad2) -> NC2
- J1 pad 20: unconnected-(J1-A15-Pad20) -> /A15
- J1 pad 21: unconnected-(J1-D0-Pad21) -> /D0
- J1 pad 22: unconnected-(J1-D1-Pad22) -> /D1
- J1 pad 23: unconnected-(J1-D2-Pad23) -> /D2
- J1 pad 24: unconnected-(J1-D3-Pad24) -> /D3
- J1 pad 25: unconnected-(J1-D4-Pad25) -> /D4
- J1 pad 26: unconnected-(J1-D5-Pad26) -> /D5
- J1 pad 27: unconnected-(J1-D6-Pad27) -> /D6
- J1 pad 28: unconnected-(J1-D7-Pad28) -> /D7
- J1 pad 29: unconnected-(J1-RW/-Pad29) -> RW/
- J1 pad 3: unconnected-(J1-NC-Pad3) -> NC3
- J1 pad 30: unconnected-(J1-NC-Pad30) -> NC30
- J1 pad 31: unconnected-(J1-BE-Pad31) -> BE
- J1 pad 32: unconnected-(J1-IRQ-Pad32) -> IRQ
- J1 pad 33: unconnected-(J1-NMI-Pad33) -> NMI
- J1 pad 34: unconnected-(J1-RES-Pad34) -> RES
- J1 pad 35: unconnected-(J1-CS/-Pad35) -> CS/
- J1 pad 36: unconnected-(J1-NC-Pad36) -> NC36
- J1 pad 37: unconnected-(J1-+5V-Pad37) -> +5V
- J1 pad 38: unconnected-(J1-NC-Pad38) -> NC38
- J1 pad 39: unconnected-(J1-CLK-Pad39) -> CLK
- J1 pad 4: unconnected-(J1-+5V-Pad4) -> +5V
- J1 pad 40: unconnected-(J1-Vss-Pad40) -> GND
- J1 pad 5: unconnected-(J1-A0-Pad5) -> /A0
- J1 pad 6: unconnected-(J1-A1-Pad6) -> /A1
- J1 pad 7: unconnected-(J1-A2-Pad7) -> /A2
- J1 pad 8: unconnected-(J1-A3-Pad8) -> /A3
- J1 pad 9: unconnected-(J1-A4-Pad9) -> /A4

Commit message: begin wiring pcb
Parts:
- removed D37, D38, D41, D43, D45, D47, D49, D51, D53, D55, D57, D59, D61, D63, D65, D67, D69, D71: Green LED, LED_THT:LED_D3.0mm
- removed D39, D40, D42, D44, D46, D48, D50, D52, D54, D56, D58, D60, D62, D64, D66, D68, D70, D72: Red LED, LED_THT:LED_D3.0mm
- removed R100, R101, R102, R103, R104, R105, R106, R107, R108, R109, R110, R111, R79, R80, R81, R82, R83, R84, R85, R86, R87, R88, R89, R90, R91, R92, R93, R94, R95, R96, R97, R98, R99: 1k, Resistor_THT:R_Axial_DIN0204_L3.6mm_D1.6mm_P2.54mm_Vertical
- added D73: Wallputer_Dual_LED, Wallputer:Wallputer_Dual_LED, F.Cu at (125.8, 109.9)
- added R35: 680, Resistor_SMD:R_0603_1608Metric, F.Cu at (75.2, 29.8)
- added R36: 680, Resistor_SMD:R_0603_1608Metric, F.Cu at (75.2, 33.0)
- added R37: 680, Resistor_SMD:R_0603_1608Metric, F.Cu at (75.2, 36.1)
- added R38: 680, Resistor_SMD:R_0603_1608Metric, F.Cu at (75.2, 39.3)
- added R39: 680, Resistor_SMD:R_0603_1608Metric, F.Cu at (75.2, 42.4)
- added R40: 680, Resistor_SMD:R_0603_1608Metric, F.Cu at (80.8, 4.64)
- added R41: 680, Resistor_SMD:R_0603_1608Metric, F.Cu at (80.8, 7.79)
- added R42: 680, Resistor_SMD:R_0603_1608Metric, F.Cu at (80.8, 10.9)
- added R43: 680, Resistor_SMD:R_0603_1608Metric, F.Cu at (80.8, 14.1)
- added R44: 680, Resistor_SMD:R_0603_1608Metric, F.Cu at (80.8, 17.2)
- added R45: 680, Resistor_SMD:R_0603_1608Metric, F.Cu at (80.8, 20.4)
- added R46: 680, Resistor_SMD:R_0603_1608Metric, F.Cu at (80.8, 23.5)
- added R47: 680, Resistor_SMD:R_0603_1608Metric, F.Cu at (80.8, 26.7)
- added R48: 680, Resistor_SMD:R_0603_1608Metric, F.Cu at (80.8, 29.8)
- added R49: 680, Resistor_SMD:R_0603_1608Metric, F.Cu at (80.8, 33.0)
- added R50: 680, Resistor_SMD:R_0603_1608Metric, F.Cu at (80.8, 36.1)
- added R51: 680, Resistor_SMD:R_0603_1608Metric, F.Cu at (80.8, 39.3)
- added R52: 680, Resistor_SMD:R_0603_1608Metric, F.Cu at (80.8, 42.4)
- added R53: 680, Resistor_SMD:R_0603_1608Metric, F.Cu at (86.4, 4.64)
- added R54: 680, Resistor_SMD:R_0603_1608Metric, F.Cu at (86.4, 7.79)
- added R55: 680, Resistor_SMD:R_0603_1608Metric, F.Cu at (86.4, 10.9)
- added R56: 680, Resistor_SMD:R_0603_1608Metric, F.Cu at (86.4, 14.1)
- added R57: 680, Resistor_SMD:R_0603_1608Metric, F.Cu at (86.4, 17.2)
- added R58: 680, Resistor_SMD:R_0603_1608Metric, F.Cu at (86.4, 20.4)
- added R59: 680, Resistor_SMD:R_0603_1608Metric, F.Cu at (86.4, 23.5)
- added R60: 680, Resistor_SMD:R_0603_1608Metric, F.Cu at (86.4, 26.7)
- added R61: 680, Resistor_SMD:R_0603_1608Metric, F.Cu at (86.4, 29.8)
- added R62: 680, Resistor_SMD:R_0603_1608Metric, F.Cu at (86.4, 33.0)
- added R63: 680, Resistor_SMD:R_0603_1608Metric, F.Cu at (86.4, 36.1)
- added R64: 680, Resistor_SMD:R_0603_1608Metric, F.Cu at (86.4, 39.3)
- added R65: 680, Resistor_SMD:R_0603_1608Metric, F.Cu at (86.4, 42.4)
- added R66: 680, Resistor_SMD:R_0603_1608Metric, F.Cu at (92.0, 4.64)
- added R67: 680, Resistor_SMD:R_0603_1608Metric, F.Cu at (92.0, 7.79)
- D1, D10, D12, D15, D17, D19, D21, D23, D25, D27, D28, D31, D33, D35, D4, D7, D9: value Green LED -> Wallputer_Dual_LED; footprint LED_THT:LED_D3.0mm -> Wallputer:Wallputer_Dual_LED
- D11, D13, D14, D16, D18, D20, D22, D24, D26, D29, D30, D32, D34, D36, D5, D6, D8: value Red LED -> Wallputer_Dual_LED; footprint LED_THT:LED_D3.0mm -> Wallputer:Wallputer_Dual_LED
- R10, R11, R12, R13, R14, R15, R16, R17, R18, R19, R20, R21, R22, R23, R24, R25, R26, R27, R28, R29, R30, R5, R6, R68, R69, R7, R70, R71, R72, R73, R74, R75, R76, R77, R78, R8, R9: value 1k -> 680; footprint Resistor_THT:R_Axial_DIN0204_L3.6mm_D1.6mm_P2.54mm_Vertical -> Resistor_SMD:R_0603_1608Metric
- U1: value NE555P -> TLC555CD
- U12, U16, U17, U18, U2, U3: footprint Package_DIP:DIP-14_W7.62mm_Socket -> Package_SO:SO-14_3.9x8.65mm_P1.27mm
- moved U2 252.7 mm to (147.4, 116.2), turned to 180 degrees
- moved U3 250.7 mm to (147.4, 135.3), turned to 180 degrees
- moved U12 235.9 mm to (147.4, 125.7), turned to 180 degrees
- moved R3 227.1 mm to (137.2, 150.5), turned to -90 degrees
- moved D32 219.9 mm to (135.0, 9.60)
- moved D31 219.5 mm to (135.0, 5.25)
- moved J1 219.0 mm to (161.3, 138.4), turned to 180 degrees
- moved D2 216.9 mm to (148.0, 149.9), turned to 180 degrees
- moved U16 216.8 mm to (147.4, 106.7), turned to 180 degrees
- moved R4 215.3 mm to (124.5, 155.5), turned to 90 degrees
- moved D17 213.0 mm to (125.7, 117.5)
- moved R33 212.1 mm to (124.5, 150.4), turned to 90 degrees
- moved D12 210.2 mm to (114.4, 13.9)
- moved D11 209.8 mm to (114.4, 9.60)
- moved D10 209.5 mm to (114.4, 5.25)
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Connections:
- D1 pad 1: Net-(D1-K) -> Net-(D1-Green_A)
- D1 pad 2: Net-(D1-A) -> Net-(D1-Red_A)
- D10 pad 1: Net-(D10-K) -> Net-(D10-Green_A)
- D10 pad 2: Net-(D10-A) -> Net-(D10-Red_A)
- D11 pad 1: Net-(D11-K) -> Net-(D11-Green_A)
- D11 pad 2: Net-(D10-K) -> Net-(D11-Red_A)
- D12 pad 1: Net-(D12-K) -> Net-(D12-Green_A)
- D12 pad 2: Net-(D12-A) -> Net-(D12-Red_A)
- D13 pad 1: Net-(D13-K) -> Net-(D13-Green_A)
- D13 pad 2: Net-(D12-K) -> Net-(D13-Red_A)
- D14 pad 1: Net-(D14-K) -> Net-(D14-Green_A)
- D14 pad 2: Net-(D14-A) -> Net-(D14-Red_A)
- D15 pad 1: Net-(D15-K) -> Net-(D15-Green_A)
- D15 pad 2: Net-(D15-A) -> Net-(D15-Red_A)
- D16 pad 1: Net-(D16-K) -> Net-(D16-Green_A)
- D16 pad 2: Net-(D15-K) -> Net-(D16-Red_A)
- D17 pad 1: Net-(D17-K) -> Net-(D17-Green_A)
- D17 pad 2: Net-(D17-A) -> Net-(D17-Red_A)
- D18 pad 1: Net-(D18-K) -> Net-(D18-Green_A)
- D18 pad 2: Net-(D17-K) -> Net-(D18-Red_A)
- D19 pad 1: Net-(D19-K) -> Net-(D19-Green_A)
- D19 pad 2: Net-(D19-A) -> Net-(D19-Red_A)
- D20 pad 1: Net-(D20-K) -> Net-(D20-Green_A)
- D20 pad 2: Net-(D19-K) -> Net-(D20-Red_A)
- D21 pad 1: Net-(D21-K) -> Net-(D21-Green_A)
- D21 pad 2: Net-(D21-A) -> Net-(D21-Red_A)
- D22 pad 1: Net-(D22-K) -> Net-(D22-Green_A)
- D22 pad 2: Net-(D21-K) -> Net-(D22-Red_A)
- D23 pad 1: Net-(D23-K) -> Net-(D23-Green_A)
- D23 pad 2: Net-(D23-A) -> Net-(D23-Red_A)
- D24 pad 1: Net-(D24-K) -> Net-(D24-Green_A)
- D24 pad 2: Net-(D23-K) -> Net-(D24-Red_A)
- D25 pad 1: Net-(D25-K) -> Net-(D25-Green_A)
- D25 pad 2: Net-(D25-A) -> Net-(D25-Red_A)
- D26 pad 1: Net-(D26-K) -> Net-(D26-Green_A)
- D26 pad 2: Net-(D25-K) -> Net-(D26-Red_A)
- D27 pad 1: Net-(D27-K) -> Net-(D27-Green_A)
- D27 pad 2: Net-(D27-A) -> Net-(D27-Red_A)
- D28 pad 1: Net-(D28-K) -> Net-(D28-Green_A)
- D29 pad 1: Net-(D29-K) -> Net-(D29-Green_A)
- D29 pad 2: Net-(D27-K) -> Net-(D29-Red_A)
- D30 pad 1: Net-(D30-K) -> Net-(D30-Green_A)
- D30 pad 2: Net-(D28-K) -> Net-(D30-Red_A)
- D31 pad 1: Net-(D31-K) -> Net-(D31-Green_A)
- D32 pad 1: Net-(D32-K) -> Net-(D32-Green_A)
- D32 pad 2: Net-(D31-K) -> Net-(D32-Red_A)
- D33 pad 1: Net-(D33-K) -> Net-(D33-Green_A)
- D34 pad 1: Net-(D34-K) -> Net-(D34-Green_A)
- D34 pad 2: Net-(D33-K) -> Net-(D34-Red_A)
- D35 pad 1: Net-(D35-K) -> Net-(D35-Green_A)
- D35 pad 2: Net-(D35-A) -> Net-(D35-Red_A)
- D36 pad 1: Net-(D36-K) -> Net-(D36-Green_A)
- D36 pad 2: Net-(D35-K) -> Net-(D36-Red_A)
- D4 pad 1: Net-(D4-K) -> Net-(D4-Green_A)
- D4 pad 2: Net-(D4-A) -> Net-(D4-Red_A)
- D5 pad 1: Net-(D5-K) -> Net-(D5-Green_A)
- D5 pad 2: Net-(D1-K) -> Net-(D5-Red_A)
- D6 pad 1: Net-(D6-K) -> Net-(D6-Green_A)
- D6 pad 2: Net-(D4-K) -> Net-(D6-Red_A)
- D7 pad 1: Net-(D7-K) -> Net-(D7-Green_A)
- D7 pad 2: Net-(D7-A) -> Net-(D7-Red_A)
- D8 pad 1: Net-(D8-K) -> Net-(D8-Green_A)
- D8 pad 2: Net-(D7-K) -> Net-(D8-Red_A)
- D9 pad 1: Net-(D14-A) -> Net-(D9-Green_A)
- D9 pad 2: Net-(D9-A) -> Net-(D9-Red_A)
- Q1 pad 2: Net-(Q1-D) -> Net-(D22-Green_K)
- R10 pad 2: Net-(D11-K) -> Net-(D7-Red_A)
- R11 pad 1: Net-(Q1-D) -> Net-(D22-Green_K)
- R11 pad 2: Net-(D12-A) -> Net-(D8-Green_K)
- R12 pad 2: Net-(D13-K) -> Net-(D8-Red_A)
- R13 pad 1: Net-(Q1-D) -> Net-(D22-Green_K)
- R13 pad 2: Net-(D27-A) -> Net-(D10-Green_K)
- R14 pad 2: Net-(D29-K) -> Net-(D10-Red_A)
- R15 pad 1: Net-(Q1-D) -> Net-(D22-Green_K)
- R15 pad 2: Net-(D1-A) -> Net-(D1-Green_K)
- R16 pad 1: Net-(Q1-D) -> Net-(D22-Green_K)
- R16 pad 2: Net-(D9-A) -> Net-(D14-Green_K)
- R17 pad 2: Net-(D14-K) -> Net-(D14-Red_A)
- R18 pad 1: Net-(Q1-D) -> Net-(D22-Green_K)
- R18 pad 2: Net-(D15-A) -> Net-(D9-Green_K)
- R19 pad 1: Net-(Q1-D) -> Net-(D22-Green_K)
- R19 pad 2: Net-(D38-A) -> Net-(D11-Green_K)
- R20 pad 2: Net-(D39-K) -> Net-(D11-Red_A)
- R21 pad 1: Net-(Q1-D) -> Net-(D22-Green_K)
- R21 pad 2: Net-(D63-A) -> Net-(D12-Green_K)
- R22 pad 2: Net-(D64-K) -> Net-(D12-Red_A)
- R23 pad 1: Net-(Q1-D) -> Net-(D22-Green_K)
- R23 pad 2: Net-(D65-A) -> Net-(D13-Green_K)
- R24 pad 2: Net-(D66-K) -> Net-(D13-Red_A)
- R25 pad 1: Net-(Q1-D) -> Net-(D22-Green_K)
- R25 pad 2: Net-(D67-A) -> Net-(D27-Green_K)
- R26 pad 2: Net-(D68-K) -> Net-(D27-Red_A)
- R27 pad 1: Net-(Q1-D) -> Net-(D22-Green_K)
- R27 pad 2: Net-(D69-A) -> Net-(D29-Green_K)
- R28 pad 2: Net-(D70-K) -> Net-(D29-Red_A)
- R29 pad 1: Net-(Q1-D) -> Net-(D22-Green_K)
- R29 pad 2: Net-(D71-A) -> Net-(D30-Green_K)
- R30 pad 2: Net-(D72-K) -> Net-(D30-Red_A)
- R5 pad 1: Net-(Q1-D) -> Net-(D22-Green_K)
- R5 pad 2: Net-(D4-A) -> Net-(D4-Green_K)
- R6 pad 2: Net-(D6-K) -> Net-(D4-Red_A)
- R68 pad 2: Net-(D16-K) -> Net-(D9-Red_A)
- R69 pad 1: Net-(Q1-D) -> Net-(D22-Green_K)
- R69 pad 2: Net-(D17-A) -> Net-(D17-Green_K)
- R7 pad 1: Net-(Q1-D) -> Net-(D22-Green_K)
- R7 pad 2: Net-(D7-A) -> Net-(D6-Green_K)
- R70 pad 2: Net-(D5-K) -> Net-(D1-Red_A)
- R71 pad 2: Net-(D18-K) -> Net-(D17-Red_A)
- R72 pad 1: Net-(Q1-D) -> Net-(D22-Green_K)
- R72 pad 2: Net-(D19-A) -> Net-(D19-Green_K)
- R73 pad 2: Net-(D20-K) -> Net-(D19-Red_A)
- R74 pad 1: Net-(Q1-D) -> Net-(D22-Green_K)
- R74 pad 2: Net-(D21-A) -> Net-(D73-Green_K)
- R75 pad 2: Net-(D22-K) -> Net-(D73-Red_A)
- R76 pad 1: Net-(Q1-D) -> Net-(Q2-D)
- R76 pad 2: Net-(D23-A) -> Net-(D35-Red_A)
- R77 pad 1: Net-(Q2-D) -> Net-(D22-Green_K)
- R77 pad 2: Net-(D24-K) -> Net-(D36-Green_K)
- R78 pad 1: Net-(Q1-D) -> Net-(Q2-D)
- R78 pad 2: Net-(D25-A) -> Net-(D36-Red_A)
- R8 pad 2: Net-(D8-K) -> Net-(D6-Red_A)
- R9 pad 1: Net-(Q1-D) -> Net-(D22-Green_K)
- R9 pad 2: Net-(D10-A) -> Net-(D7-Green_K)
- U12 pad 10: Net-(D14-A) -> Net-(D14-Green_A)
- U12 pad 12: Net-(D61-K) -> Net-(D28-Green_A)
- U12 pad 2: Net-(D59-K) -> Net-(D26-Green_A)
- U12 pad 4: Net-(D1-K) -> Net-(D1-Green_A)
- U12 pad 6: Net-(D15-K) -> Net-(D9-Green_A)
- U12 pad 8: Net-(D17-K) -> Net-(D17-Green_A)
- U16 pad 10: Net-(D25-K) -> Net-(D15-Green_A)
- U16 pad 12: Net-(D21-K) -> Net-(D73-Green_A)
- U16 pad 2: Net-(D19-K) -> Net-(D19-Green_A)
- U16 pad 4: Net-(D23-K) -> Net-(D5-Green_A)
- U16 pad 6: Net-(D28-K) -> Net-(D16-Green_A)
- U16 pad 8: Net-(D31-K) -> Net-(D18-Green_A)
- U17 pad 10: Net-(D41-K) -> Net-(D32-Green_A)
- U17 pad 12: Net-(D35-K) -> Net-(D21-Green_A)
- U17 pad 2: Net-(D33-K) -> Net-(D20-Green_A)
- U17 pad 4: Net-(D37-K) -> Net-(D31-Green_A)
- U17 pad 6: Net-(D43-K) -> Net-(D33-Green_A)
- U17 pad 8: Net-(D45-K) -> Net-(D34-Green_A)
- U18 pad 10: Net-(D53-K) -> Net-(D23-Green_A)
- U18 pad 12: Net-(D49-K) -> Net-(D36-Green_A)
- U18 pad 2: Net-(D47-K) -> Net-(D35-Green_A)
- U18 pad 4: Net-(D51-K) -> Net-(D22-Green_A)
- U18 pad 6: Net-(D55-K) -> Net-(D24-Green_A)
- U18 pad 8: Net-(D57-K) -> Net-(D25-Green_A)
- U2 pad 10: Net-(D7-K) -> Net-(D6-Green_A)
- U2 pad 12: Net-(D38-K) -> Net-(D11-Green_A)
- U2 pad 13: NC2 -> NC3
- U2 pad 2: Net-(D27-K) -> Net-(D10-Green_A)
- U2 pad 4: Net-(D4-K) -> Net-(D4-Green_A)
- U2 pad 6: Net-(D10-K) -> Net-(D7-Green_A)
- U2 pad 8: Net-(D12-K) -> Net-(D8-Green_A)
- U3 pad 10: Net-(D65-K) -> Net-(D13-Green_A)
- U3 pad 11: NC30 -> NC38
- U3 pad 2: Net-(D71-K) -> Net-(D30-Green_A)
- U3 pad 3: NC3 -> NC2
- U3 pad 4: Net-(D63-K) -> Net-(D12-Green_A)
- U3 pad 5: NC36 -> NC3
- U3 pad 6: Net-(D67-K) -> Net-(D27-Green_A)
- U3 pad 8: Net-(D69-K) -> Net-(D29-Green_A)
- U3 pad 9: NC38 -> NC36
Routing:
- net +5V: track 0.00 -> 261.7 mm, vias 0 -> 6
- net Net-(Q2-D): track 0.00 -> 39.2 mm
- net Net-(R32-Pad1): track 0.00 -> 38.3 mm, vias 0 -> 1
- net SW_BUS_LED: track 0.00 -> 33.6 mm
- net Net-(D22-Green_K): track 0.00 -> 32.8 mm
- net Net-(U1-THR): track 0.00 -> 26.5 mm
- net GND: track 0.00 -> 21.8 mm, vias 0 -> 6
- net NC36: track 0.00 -> 18.2 mm
- net NC38: track 0.00 -> 17.2 mm
- net NC2: track 0.00 -> 15.3 mm
- net NC3: track 0.00 -> 15.2 mm
- net RES: track 0.00 -> 13.6 mm
- net CLK: track 0.00 -> 12.7 mm
- net Net-(D2-A): track 0.00 -> 8.74 mm
- net SW_BUS_LEDb: track 0.00 -> 6.37 mm
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- added copper zone on B.Cu, net GND
- added copper zone on F.Cu, net GND
Other:
- board text added: "A0"
- board text added: "A1"
- board text added: "A10"
- board text added: "A11"
- board text added: "A12"
- board text added: "A13"
- board text added: "A14"
- board text added: "A15"
- board text added: "A2"
- board text added: "A3"
- board text added: "A4"
- board text added: "A5"
- board text added: "A6"
- board text added: "A7"
- board text added: "A8"
- board text added: "A9"

Commit message: More layout
Parts:
- moved R15 132.7 mm to (130.4, 125.7), turned to 180 degrees
- moved R16 126.5 mm to (130.4, 121.9), turned to 180 degrees
- moved D1 121.2 mm to (125.7, 125.1)
- moved R21 119.5 mm to (130.4, 129.5), turned to 180 degrees
- moved R17 118.4 mm to (121.3, 120.7)
- moved R18 117.8 mm to (130.4, 118.1), turned to 180 degrees
- moved D12 115.5 mm to (125.7, 128.9)
- moved D27 114.4 mm to (125.7, 132.7)
- moved R25 112.0 mm to (130.4, 133.3), turned to 180 degrees
- moved C22 111.8 mm to (144.7, 142.9), turned to 180 degrees
- moved R22 111.1 mm to (121.1, 128.3)
- moved R68 109.8 mm to (121.1, 116.8)
- moved D4 109.0 mm to (91.4, 117.4)
- moved C21 107.4 mm to (153.0, 129.5), turned to 90 degrees
- moved R5 105.8 mm to (96.1, 118.1), turned to 180 degrees
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Connections:
- Q1 pad 2: Net-(D22-Green_K) -> Net-(Q1-D)
- R11 pad 1: Net-(D22-Green_K) -> Net-(Q1-D)
- R13 pad 1: Net-(D22-Green_K) -> Net-(Q1-D)
- R15 pad 1: Net-(D22-Green_K) -> Net-(Q1-D)
- R16 pad 1: Net-(D22-Green_K) -> Net-(Q1-D)
- R18 pad 1: Net-(D22-Green_K) -> Net-(Q1-D)
- R19 pad 1: Net-(D22-Green_K) -> Net-(Q1-D)
- R21 pad 1: Net-(D22-Green_K) -> Net-(Q1-D)
- R23 pad 1: Net-(D22-Green_K) -> Net-(Q1-D)
- R25 pad 1: Net-(D22-Green_K) -> Net-(Q1-D)
- R27 pad 1: Net-(D22-Green_K) -> Net-(Q1-D)
- R29 pad 1: Net-(D22-Green_K) -> Net-(Q1-D)
- R35 pad 1: Net-(D22-Green_K) -> Net-(Q1-D)
- R37 pad 1: Net-(D22-Green_K) -> Net-(Q1-D)
- R39 pad 1: Net-(D22-Green_K) -> Net-(Q1-D)
- R41 pad 1: Net-(D22-Green_K) -> Net-(Q1-D)
- R43 pad 1: Net-(D22-Green_K) -> Net-(Q1-D)
- R45 pad 1: Net-(D22-Green_K) -> Net-(Q1-D)
- R47 pad 1: Net-(D22-Green_K) -> Net-(Q1-D)
- R49 pad 1: Net-(D22-Green_K) -> Net-(Q1-D)
- R5 pad 1: Net-(D22-Green_K) -> Net-(Q1-D)
- R51 pad 1: Net-(D22-Green_K) -> Net-(Q1-D)
- R53 pad 1: Net-(D22-Green_K) -> Net-(Q1-D)
- R55 pad 1: Net-(D22-Green_K) -> Net-(Q1-D)
- R57 pad 1: Net-(D22-Green_K) -> Net-(Q1-D)
- R59 pad 1: Net-(D22-Green_K) -> Net-(Q1-D)
- R61 pad 1: Net-(D22-Green_K) -> Net-(Q1-D)
- R63 pad 1: Net-(D22-Green_K) -> Net-(Q1-D)
- R65 pad 1: Net-(D22-Green_K) -> Net-(Q1-D)
- R67 pad 1: Net-(D22-Green_K) -> Net-(Q1-D)
- R69 pad 1: Net-(D22-Green_K) -> Net-(Q1-D)
- R7 pad 1: Net-(D22-Green_K) -> Net-(Q1-D)
- R72 pad 1: Net-(D22-Green_K) -> Net-(Q1-D)
- R74 pad 1: Net-(D22-Green_K) -> Net-(Q1-D)
- R77 pad 1: Net-(D22-Green_K) -> Net-(Q1-D)
- R9 pad 1: Net-(D22-Green_K) -> Net-(Q1-D)
Routing:
- net Net-(Q1-D): track 0.00 -> 170.0 mm, vias 0 -> 2
- net Net-(Q2-D): track 39.2 -> 177.5 mm
- net Net-(D22-Green_K): track 32.8 -> 2.11 mm
- net Net-(D28-Green_A): track 0.00 -> 4.53 mm
- net Net-(D25-Green_A): track 0.00 -> 4.53 mm
- net Net-(D7-Green_A): track 0.00 -> 4.08 mm
- net Net-(D6-Green_A): track 0.00 -> 4.08 mm
- net Net-(D5-Green_A): track 0.00 -> 4.08 mm
- net Net-(D4-Green_A): track 0.00 -> 4.08 mm
- net Net-(D32-Green_A): track 0.00 -> 4.08 mm
- net Net-(D31-Green_A): track 0.00 -> 4.08 mm
- net Net-(D30-Green_A): track 0.00 -> 4.08 mm
- net Net-(D29-Green_A): track 0.00 -> 4.08 mm
- net Net-(D27-Green_A): track 0.00 -> 4.08 mm
- net Net-(D24-Green_A): track 0.00 -> 4.08 mm
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Other:
- board text added: "BE"
- board text added: "CLK"
- board text added: "CS/"
- board text added: "D0"
- board text added: "D1"
- board text added: "D2"
- board text added: "D3"
- board text added: "D4"
- board text added: "D5"
- board text added: "D6"
- board text added: "D7"
- board text added: "IRQ/"
- board text added: "NC2"
- board text added: "NC3"
- board text added: "NC30"
- board text added: "NC36"
- board text added: "NC38"
- board text added: "NMI/"
- board text added: "RW/"
