File: wallputer-modular/memory-card/memory-card.kicad_sch (KiCad schematic)
At the start: 8 parts, among them U1 HM62256BLP, U2 74HC00, U3 SST39SF010

Commit message: add activation indicators
Parts:
- added D1, D2: Blue, LED_SMD:LED_1206_3216Metric, symbol Device:LED
- added Q1, Q2: BSS84, Package_TO_SOT_SMD:SOT-23, symbol Transistor_FET:BSS84
- added R2, R7: 680, Resistor_SMD:R_0603_1608Metric, symbol Device:R
- added R3, R5: 5.1k, Resistor_SMD:R_0603_1608Metric, symbol Device:R
- added R4, R6: 100k, Resistor_SMD:R_0603_1608Metric, symbol Device:R
Connections:
- net +5V: now also Q1.2 (S), Q2.2 (S), R4.2, R6.2
- net GND: now also D1.1 (K), D2.1 (K)
- net RAM/: now also R3.2
- net ROM/: now also R5.2
- new net: D1.2 (A), R2.1
- new net: D2.2 (A), R7.1
- new net: Q1.1 (G), R3.1, R4.1
- new net: Q1.3 (D), R2.2
- new net: Q2.1 (G), R5.1, R6.1
- new net: Q2.3 (D), R7.2
