File: wallputer-modular/clock-card/clock-card.kicad_pcb (KiCad board)
At the start: 2 copper layers, 99.7 x 99.7 mm, 1 part

Commit message: finish design for clock card
Parts:
- added C1: 10uF, Capacitor_THT:CP_Radial_D5.0mm_P2.00mm, F.Cu at (95.2, 144.8)
- added C10: 10uF, Capacitor_THT:CP_Radial_D5.0mm_P2.00mm, F.Cu at (69.2, 128.8)
- added C11: 100nF, Capacitor_THT:C_Disc_D5.0mm_W2.5mm_P5.00mm, F.Cu at (123.2, 134.0)
- added C12: 100nF, Capacitor_THT:C_Disc_D5.0mm_W2.5mm_P5.00mm, F.Cu at (118.7, 61.6)
- added C2: 103, Capacitor_THT:C_Disc_D5.0mm_W2.5mm_P5.00mm, F.Cu at (100.3, 129.5)
- added C3: 100nF, Capacitor_THT:C_Disc_D5.0mm_W2.5mm_P5.00mm, F.Cu at (86.4, 76.2)
- added C4: 100nF, Capacitor_THT:C_Disc_D5.0mm_W2.5mm_P5.00mm, F.Cu at (138.4, 111.5)
- added C5: 100nF, Capacitor_THT:C_Disc_D5.0mm_W2.5mm_P5.00mm, F.Cu at (89.3, 132.2)
- added C6: 100nF, Capacitor_THT:C_Disc_D5.0mm_W2.5mm_P5.00mm, F.Cu at (69.8, 116.2)
- added C7: 103, Capacitor_THT:C_Disc_D5.0mm_W2.5mm_P5.00mm, F.Cu at (66.0, 121.9)
- added C8: 100nF, Capacitor_THT:C_Disc_D5.0mm_W2.5mm_P5.00mm, F.Cu at (105.4, 141.6)
- added C9: 100nF, Capacitor_THT:C_Disc_D5.0mm_W2.5mm_P5.00mm, F.Cu at (73.7, 133.3)
- added D1: Red / MHz, LED_THT:LED_D1.8mm_W3.3mm_H2.4mm, F.Cu at (128.9, 95.9)
- added D2: Yellow / kHz, LED_THT:LED_D1.8mm_W3.3mm_H2.4mm, F.Cu at (128.9, 92.1)
- added D3: Green / Hz, LED_THT:LED_D1.8mm_W3.3mm_H2.4mm, F.Cu at (128.9, 88.3)
- added J2: ICP, Connector_PinHeader_2.54mm:PinHeader_1x04_P2.54mm_Vertical, F.Cu at (125.1, 67.9)
- added Q2: BSS84, Package_TO_SOT_SMD:SOT-23, F.Cu at (120.7, 83.5)
- added Q4: BSS84, Package_TO_SOT_SMD:SOT-23, F.Cu at (109.9, 83.5)
- added Q6: BSS84, Package_TO_SOT_SMD:SOT-23, F.Cu at (98.7, 83.5)
- added R1: 1k, Resistor_THT:R_Axial_DIN0204_L3.6mm_D1.6mm_P2.54mm_Vertical, F.Cu at (95.2, 129.5)
- added R11: 100k, Resistor_SMD:R_0603_1608Metric, F.Cu at (110.0, 80.7)
- added R14: 100k, Resistor_SMD:R_0603_1608Metric, F.Cu at (98.9, 80.6)
- added R15: 330, Resistor_SMD:R_0603_1608Metric, F.Cu at (113.7, 75.1)
- added R16: 330, Resistor_SMD:R_0603_1608Metric, F.Cu at (115.6, 75.1)
- added R17: 330, Resistor_SMD:R_0603_1608Metric, F.Cu at (117.5, 75.1)
- added R18: 330, Resistor_SMD:R_0603_1608Metric, F.Cu at (106.0, 75.1)
- added R19: 330, Resistor_SMD:R_0603_1608Metric, F.Cu at (108.0, 75.1)
- added R2: 10k, Resistor_THT:R_Axial_DIN0204_L3.6mm_D1.6mm_P2.54mm_Vertical, F.Cu at (125.1, 111.5)
- added R20: 330, Resistor_SMD:R_0603_1608Metric, F.Cu at (109.9, 75.1)
- added R21: 330, Resistor_SMD:R_0603_1608Metric, F.Cu at (111.8, 75.1)
- added R22: 330, Resistor_SMD:R_0603_1608Metric, F.Cu at (104.1, 75.1)
- added R3: 1k, Resistor_THT:R_Axial_DIN0204_L3.6mm_D1.6mm_P2.54mm_Vertical, F.Cu at (92.7, 127.0)
- added R4: 10k, Resistor_THT:R_Axial_DIN0204_L3.6mm_D1.6mm_P2.54mm_Vertical, F.Cu at (83.3, 114.0)
- added R5: 1M, Resistor_THT:R_Axial_DIN0204_L3.6mm_D1.6mm_P2.54mm_Vertical, F.Cu at (71.1, 125.1)
- added R6: 1k, Resistor_SMD:R_0603_1608Metric, F.Cu at (147.8, 95.9)
- added R7: 1k, Resistor_SMD:R_0603_1608Metric, F.Cu at (147.8, 92.1)
- added R8: 100k, Resistor_SMD:R_0603_1608Metric, F.Cu at (120.8, 80.7)
- added R9: 1k, Resistor_SMD:R_0603_1608Metric, F.Cu at (147.8, 88.3)
- added RV1: 1M, Potentiometer_THT:Potentiometer_Alpha_RD901F-40-00D_Single_Vertical, F.Cu at (92.8, 121.3)
- added SW1: switch clock, Button_Switch_THT:SW_PUSH_6mm_H4.3mm, F.Cu at (134.6, 115.9)
- added SW2: step, Button_Switch_THT:SW_PUSH_6mm_H4.3mm, F.Cu at (73.7, 111.7)
- added U1: 74HC14, Package_DIP:DIP-14_W7.62mm_Socket, F.Cu at (82.5, 73.7)
- added U2: NE555P, Package_DIP:DIP-8_W7.62mm, F.Cu at (92.7, 139.7)
- added U3: 74HC93, Package_DIP:DIP-14_W7.62mm_Socket, F.Cu at (109.2, 131.4)
- added U4: NE555P, Package_DIP:DIP-8_W7.62mm, F.Cu at (81.3, 130.2)
- added U5: 74HC153, Package_DIP:DIP-16_W7.62mm_Socket, F.Cu at (126.4, 141.6)
- added U6: ATtiny1616-S, Package_SO:SOIC-20W_7.5x12.8mm_P1.27mm, F.Cu at (110.5, 66.5)
- added U7: INND-TS40, Wallputer:INND-TS40, F.Cu at (120.7, 92.1)
- added U8: INND-TS40, Wallputer:INND-TS40, F.Cu at (109.9, 92.1)
- added U9: INND-TS40, Wallputer:INND-TS40, F.Cu at (99.1, 92.1)
- added Y1: 1 MHz, Oscillator:Oscillator_DIP-14, F.Cu at (109.9, 110.5)
- moved J1 94.5 mm to (137.8, 151.2), turned to -90 degrees
Connections:
- J1 pad 39: unconnected-(J1-CLK-Pad39) -> CLK
Routing:
- net +5V: track 2.54 -> 339.2 mm, vias 0 -> 3
- net CLK: track 0.00 -> 123.9 mm, vias 0 -> 1
- net Net-(U3-~{CKA}): track 0.00 -> 82.7 mm
- net Net-(C4-Pad1): track 0.00 -> 80.3 mm
- net Net-(U4-Q): track 0.00 -> 73.3 mm
- net Net-(U6-PA5): track 0.00 -> 70.4 mm
- net Net-(U6-PA6): track 0.00 -> 66.6 mm
- net Net-(U6-PA7): track 0.00 -> 62.5 mm
- net Net-(U4-TR): track 0.00 -> 59.8 mm
- net Net-(C6-Pad1): track 0.00 -> 58.7 mm
- net Net-(U6-PB2): track 0.00 -> 46.7 mm
- net Net-(U7-G): track 0.00 -> 45.7 mm
- net Net-(U7-D): track 0.00 -> 45.4 mm
- net Net-(U7-C): track 0.00 -> 44.6 mm
- net Net-(U7-DP): track 0.00 -> 43.9 mm
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Other:
- board text added: "1MHz"
- board text added: "CARD"
- board text added: "CLOCK"
- board text added: "Hz"
- board text added: "MHz"
- board text added: "SINGLE STEP"
- board text added: "SWITCH SOURCE"
- board text added: "VARIABLE"
- board text added: "kHz"

Commit message: improve design a little
Parts:
- added R10: 68, Resistor_SMD:R_0603_1608Metric, F.Cu at (146.7, 139.3)
Connections:
- C6 pad 2: GND -> +5V
- R4 pad 1: +5V -> GND
- SW2 pad 1: GND -> +5V
- U1 pad 13: CLK -> Net-(R10-Pad2)
Routing:
- net Net-(R10-Pad2): track 0.00 -> 106.3 mm, vias 0 -> 1
- net CLK: track 123.9 -> 18.0 mm, vias 1 -> 0
- net +5V: track 339.2 -> 352.2 mm
Other:
- board text added: "+5V"
- board text added: "GND"
- board text added: "IC Vdd"
- board text added: "ICP"
