File: wallputer-modular/clock-card/clock-card.kicad_sch (KiCad schematic)
At the start: 1 part

Commit message: initial design for clock card
Parts:
- added C1, C6: 103, Capacitor_THT:C_Disc_D5.0mm_W2.5mm_P5.00mm, symbol Device:C
- added C10, C11, C12, C2, C3, C4, C5, C7, C8: 100nF, Capacitor_THT:C_Disc_D5.0mm_W2.5mm_P5.00mm, symbol Device:C
- added C9: 10uF, Capacitor_THT:CP_Radial_D5.0mm_P2.00mm, symbol Device:C_Polarized
- added D1: Red / MHz, LED_THT:LED_D1.8mm_W3.3mm_H2.4mm, symbol Device:LED
- added D2: Yellow / kHz, LED_THT:LED_D1.8mm_W3.3mm_H2.4mm, symbol Device:LED
- added D3: Green / Hz, LED_THT:LED_D1.8mm_W3.3mm_H2.4mm, symbol Device:LED
- added Q1, Q2, Q3: BC847, Package_TO_SOT_SMD:SOT-23, symbol Transistor_BJT:BC847
- added R1, R3: 1k, Resistor_THT:R_Axial_DIN0204_L3.6mm_D1.6mm_P2.54mm_Vertical, symbol Device:R
- added R10, R11, R12, R6, R7, R8, R9: R, symbol Device:R
- added R2, R4: 10k, Resistor_THT:R_Axial_DIN0204_L3.6mm_D1.6mm_P2.54mm_Vertical, symbol Device:R
- added R5: 1m, Resistor_THT:R_Axial_DIN0204_L3.6mm_D1.6mm_P2.54mm_Vertical, symbol Device:R
- added RV1: 1M, Potentiometer_THT:Potentiometer_Alpha_RD901F-40-00D_Single_Vertical, symbol Device:R_Potentiometer
- added SW1: switch clock, Button_Switch_THT:SW_PUSH_6mm_H4.3mm, symbol Switch:SW_Push
- added SW2: step, Button_Switch_THT:SW_PUSH_6mm_H4.3mm, symbol Switch:SW_Push
- added U1: 74HC14, Package_DIP:DIP-14_W7.62mm_Socket, symbol 74xx:74HC14
- added U10, U8, U9: INND-TS40, Wallputer:INND-TS40, symbol Wallputer:INND-TS40_1
- added U2, U4: NE555P, Package_DIP:DIP-8_W7.62mm, symbol Timer:NE555P
- added U3: 74HC93, Package_DIP:DIP-14_W7.62mm_Socket, symbol 74xx_IEEE:7493
- added U5: 74HC153, Package_DIP:DIP-16_W7.62mm_Socket, symbol 74xx_IEEE:74153
- added U6: ATtiny1616-S, Package_SO:SOIC-20W_7.5x12.8mm_P1.27mm, symbol MCU_Microchip_ATtiny:ATtiny1616-S
- added U7: MAX7219, symbol Driver_LED:MAX7219
- added Y1: 1 MHz, Oscillator:Oscillator_DIP-14, symbol Oscillator:OCXO-14
- J1: footprint Wallputer:Wallputer_Bus_Header -> Wallputer:Wallputer_Bus_*
Connections:
- net +5V: now also C10.1, C11.1, C12.1, C2.2, C4.1, C7.1, C8.1, R10.1, R12.1, R2.2, R3.2, R4.1, R5.2, R7.1, U1.14 (VCC), U2.4 (R), U2.8 (VCC), U3.5 (VCC), U4.4 (R), U4.8 (VCC), U5.16 (VCC), U6.1 (VCC), U7.19 (V+), Y1.14 (Vcc)
- net GND: now also C1.2, C10.2, C11.2, C12.2, C2.1, C3.2, C4.2, C5.2, C6.1, C7.2, C8.2, C9.2, Q1.2 (E), Q2.2 (E), Q3.2 (E), R6.1, RV1.3, SW1.1, SW2.1, U1.11, U1.5, U1.7 (GND), U1.9, U2.1 (GND), U2.2 (TR), U2.6 (THR), U3.10 (GND), U4.1 (GND), U5.1 (~{ENa}), U5.3 (I3a), U5.8 (GND), U6.20 (GND), U7.4 (GND), U7.9 (GND), Y1.7 (GND)
- net CLK: now reaches J1.39 (CLK)
- net CLK: now also U1.13, U5.7 (Qa)
- new net: R9.1, U6.10 (PB1)
- new net: Q2.1 (B), R9.2
- new net: C5.1, R4.2, SW2.2, U1.3
- new net: C9.1, R5.1, U4.6 (THR), U4.7 (DIS)
- new net: R6.2, U7.18 (ISET)
- new net: R11.1, U6.9 (PB2)
- new net: Q3.1 (B), R11.2
- new net: D2.2 (A), R10.2
- new net: U1.12, U6.2 (PA4)
- new net: Q1.1 (B), R8.2
- new net: D1.1 (K), Q1.3 (C)
- new net: U10.1 (E), U7.21 (SEG_E), U8.1 (E), U9.1 (E)
- new net: U10.10 (A), U7.14 (SEG_A), U8.10 (A), U9.10 (A)
- new net: U10.2 (F), U7.15 (SEG_F), U8.2 (F), U9.2 (F)
- new net: U10.3 (G), U7.11 (DIG_1), U7.17 (SEG_G), U8.3 (G), U9.3 (G), U9.6 (CC)
- new net: U10.5 (D), U7.23 (SEG_D), U8.5 (D), U9.5 (D)
- new net: U7.2 (DIG_0), U8.6 (CC)
- new net: U10.7 (DP), U7.22 (SEG_DP), U8.7 (DP), U9.7 (DP)
- new net: U10.8 (C), U7.20 (SEG_C), U8.8 (C), U9.8 (C)
- new net: U10.9 (B), U7.16 (SEG_B), U8.9 (B), U9.9 (B)
- new net: U2.3 (Q), U5.5 (I1a)
- new net: C1.1, U2.5 (CV)
- new net: R1.1, R3.1, U2.7 (DIS)
- new net: U5.6 (I0a), Y1.8 (OUT)
- new net: D3.2 (A), R12.2
- new net: U1.4, U4.2 (TR)
- new net: U4.3 (Q), U5.4 (I2a)
- new net: C6.2, U4.5 (CV)
- new net: C3.1, R2.1, SW1.2, U1.1
- new net: D3.1 (K), Q3.3 (C)
- new net: D1.2 (A), R7.2
- new net: U10.6 (CC), U7.6 (DIG_2)
- new net: R8.1, U6.11 (PB0)
- new net: U6.3 (PA5), U7.12 (LOAD)
- new net: U6.4 (PA6), U7.13 (CLK)
- new net: U6.5 (PA7), U7.1 (DIN)
- new net: U1.2, U3.14 (~{CKA})
- new net: D2.1 (K), Q2.3 (C)
- new net: U3.1 (~{CKB}), U3.12 (Q0), U3.2 (R0(1)), U5.14 (A)
- new net: U3.3 (R0(2)), U3.9 (Q1), U5.2 (B)
- new net: R1.2, RV1.2
- no-connect marks 0 -> 48

Commit message: finish design for clock card
Parts:
- removed C12: 100nF, Capacitor_THT:C_Disc_D5.0mm_W2.5mm_P5.00mm, symbol Device:C
- removed Q1, Q2, Q3: BC847, Package_TO_SOT_SMD:SOT-23, symbol Transistor_BJT:BC847
- removed R10, R12: R, symbol Device:R
- removed U7: MAX7219, symbol Driver_LED:MAX7219
- added C1: 10uF, Capacitor_THT:CP_Radial_D5.0mm_P2.00mm, symbol Device:C_Polarized
- added J2: ICP, Connector_PinHeader_2.54mm:PinHeader_1x04_P2.54mm_Vertical, symbol Connector:Conn_01x04_Pin
- added Q2, Q4, Q6: BSS84, Package_TO_SOT_SMD:SOT-23, symbol Transistor_FET:BSS84
- added R14: 100k, Resistor_SMD:R_0603_1608Metric, symbol Device:R
- added R15, R16, R17, R18, R19, R20, R21, R22: 330, Resistor_SMD:R_0603_1608Metric, symbol Device:R
- R11, R8: value R -> 100k; footprint (none) -> Resistor_SMD:R_0603_1608Metric
- R5: value 1m -> 1M
- R6, R7, R9: value R -> 1k; footprint (none) -> Resistor_SMD:R_0603_1608Metric
- renumbered C9 to C10, C10 to C11, C11 to C12, C1 to C2, C2 to C3, C3 to C4, C4 to C5, C5 to C6, C6 to C7, C7 to C8, C8 to C9, U8 to U7, U9 to U8, U10 to U9
Connections:
- net +5V: now also R11.1, R8.1, J2.4 (Pin_4), Q2.2 (S), Q4.2 (S), Q6.2 (S), R14.1; no longer C12.1, R7.1, U6.1 (VCC)
- net GND: now also D1.1 (K), D2.1 (K), D3.1 (K), C1.2, J2.2 (Pin_2); no longer R6.1, RV1.3, U2.2 (TR), U2.6 (THR)
- net at R9.1: now also D3.2 (A); no longer U6.10 (PB1)
- net at R9.2: now also U6.5 (PA7)
- net at R6.2: now also U6.3 (PA5)
- net at U6.9 (PB2): now also U1.12; no longer R11.1
- net at R11.2: now also U6.7 (PB4), Q4.1 (G)
- net at D2.2 (A): now also R7.1
- net at U6.2 (PA4): no longer U1.12
- net at R8.2: now also U6.6 (PB5), Q2.1 (G)
- net at U7.1 (E), U8.1 (E), U9.1 (E): now also R19.2
- net at U7.10 (A), U8.10 (A), U9.10 (A): now also R15.2
- net at U7.2 (F), U8.2 (F), U9.2 (F): now also R20.2
- net at U7.3 (G), U8.3 (G), U9.3 (G): now also R21.2; no longer U8.6 (CC)
- net at U7.5 (D), U8.5 (D), U9.5 (D): now also R18.2
- net at U7.6 (CC): now also Q2.3 (D)
- net at U7.7 (DP), U8.7 (DP), U9.7 (DP): now also R22.2
- net at U7.8 (C), U8.8 (C), U9.8 (C): now also R17.2
- net at U7.9 (B), U8.9 (B), U9.9 (B): now also R16.2
- net at U2.3 (Q): now also U5.4 (I2a); no longer U5.5 (I1a)
- net at U4.3 (Q): now also U5.5 (I1a); no longer U5.4 (I2a)
- net at D1.2 (A): now also R6.1; no longer R7.2
- net at U9.6 (CC): now also Q6.3 (D)
- net at U6.11 (PB0): now also R22.1; no longer R8.1
- net at U6.12 (PC0): now also R18.1
- net at U6.13 (PC1): now also R19.1
- net at U6.14 (PC2): now also R20.1
- net at U6.15 (PC3): now also R21.1
- net at U6.16 (~{RESET}/PA0): now also J2.1 (Pin_1)
- net at U6.17 (PA1): now also R15.1
- net at U6.18 (PA2): now also R16.1
- net at U6.19 (PA3): now also R17.1
- net at U6.4 (PA6): now also R7.2
- net at U6.8 (PB3): now also Q6.1 (G), R14.2
- new net: Q4.3 (D), U8.6 (CC)
- new net: C1.1, RV1.3, U2.2 (TR), U2.6 (THR)
- new net: C12.1, J2.3 (Pin_3), U6.1 (VCC)
- no-connect marks 48 -> 51
Other:
- note added: "Jumper on pins 3 and 4 for normal use. Remove jumper for programming"
- moved on the sheet: C12, D1, D2, D3, RV1, U1C, U1D, U1E, U1F, U6, U7, U8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

Commit message: improve design a little
Parts:
- added R10: 68, Resistor_SMD:R_0603_1608Metric, symbol Device:R
Connections:
- net +5V: now also C6.2, SW2.1; no longer R4.1
- net CLK: now also R10.1; no longer U1.13
- net GND: now also R4.1; no longer C6.2, SW2.1
- new net: R10.2, U1.13
- no-connect marks 51 -> 53
Changed lines of the file:
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@@
 	)
 	(junction
-		(at 77.47 104.14)
-		(diameter 0)
-		(color 0 0 0 0)
-	)
-	(junction
 		(at 204.47 142.24)
 		(diameter 0)
@@
 	)
 	(junction
+		(at 77.47 104.14)
+		(diameter 0)
+		(color 0 0 0 0)
+	)
+	(junction
 		(at 29.21 82.55)
 		(diameter 0)
@@
 	)
 	(junction
-		(at 81.28 109.22)
+		(at 207.01 144.78)
 		(diameter 0)
 		(color 0 0 0 0)
 	)
 	(junction
-		(at 207.01 144.78)
+		(at 81.28 109.22)
 		(diameter 0)
 		(color 0 0 0 0)
@@
 	)
 	(junction
-		(at 261.62 158.75)
+		(at 76.2 109.22)
 		(diameter 0)
 		(color 0 0 0 0)
 	)
 	(junction
-		(at 234.95 160.02)
+		(at 261.62 158.75)
 		(diameter 0)
 		(color 0 0 0 0)
 	)
 	(junction
-		(at 132.08 110.49)
+		(at 234.95 160.02)
 		(diameter 0)
 		(color 0 0 0 0)
 	)
 	(junction
-		(at 76.2 109.22)
+		(at 132.08 110.49)
 		(diameter 0)
 		(color 0 0 0 0)
@@
 	)
 	(no_connect
+		(at 180.34 151.13)
+	)
+	(no_connect
 		(at 20.32 157.48)
 	)
@@
 	)
 	(no_connect
+		(at 180.34 135.89)
+	)
+	(no_connect
 		(at 36.83 162.56)
 	)
@@
 	(wire
 		(pts
+			(xy 81.28 106.68) (xy 81.28 109.22)
+		)
+		(stroke
+			(width 0)
+			(type default)
+		)
+	)
+	(wire
+		(pts
 			(xy 184.15 140.97) (xy 184.15 149.86)
 		)
@@
 	(wire
 		(pts
-			(xy 261.62 158.75) (xy 261.62 163.83)
+			(xy 73.66 106.68) (xy 81.28 106.68)
 		)
 		(stroke
@@
 	(wire
 		(pts
-			(xy 73.66 104.14) (xy 77.47 104.14)
+			(xy 261.62 158.75) (xy 261.62 163.83)
 		)
 		(stroke
@@
 	(wire
 		(pts
-			(xy 76.2 109.22) (xy 81.28 109.22)
-		)
-		(stroke
-			(width 0)
-			(type default)
-		)
-	)
-	(wire
-		(pts
 			(xy 15.24 106.68) (xy 15.24 110.49)
 		)
@@
 	(wire
 		(pts
+			(xy 76.2 109.22) (xy 76.2 104.14)
+		)
+		(stroke
+			(width 0)
+			(type default)
+		)
+	)
+	(wire
+		(pts
 			(xy 45.72 50.8) (xy 45.72 52.07)
 		)
@@
 	(wire
 		(pts
+			(xy 73.66 104.14) (xy 73.66 106.68)
+		)
+		(stroke
+			(width 0)
+			(type default)
+		)
+	)
+	(wire
+		(pts
 			(xy 238.76 100.33) (xy 242.57 100.33)
 		)
@@
 	(wire
 		(pts
+			(xy 76.2 104.14) (xy 77.47 104.14)
+		)
+		(stroke
+			(width 0)
+			(type default)
+		)
+	)
+	(wire
+		(pts
 			(xy 55.88 92.71) (xy 55.88 90.17)
 		)
@@
 	(global_label "CLK"
 		(shape input)
-		(at 137.16 134.62 90)
+		(at 129.54 134.62 180)
 		(fields_autoplaced yes)
 		(effects
@@
 				(size 1.27 1.27)
 			)
-			(justify left)
+			(justify right)
 		)
 		(property "Intersheetrefs" "${INTERSHEET_REFS}"
-			(at 137.16 128.0667 90)
+			(at 122.9867 134.62 0)
 			(effects
 				(font
 					(size 1.27 1.27)
 				)
-				(justify left)
+				(justify right)
 				(hide yes)
 			)
@@
 					(unit 1)
 				)
+			)
+		)
+	)
+	(symbol
+		(lib_id "Device:R")
+		(at 133.35 134.62 90)
+		(unit 1)
+		(exclude_from_sim no)
+		(in_bom yes)
+		(on_board yes)
+		(dnp no)
+		(fields_autoplaced yes)
+		(property "Reference" "R10"
+			(at 132.0799 132.08 0)
+			(effects
+				(font
+					(size 1.27 1.27)
+				)
+				(justify left)
+			)
+		)
+		(property "Value" "68"
+			(at 134.6199 132.08 0)
+			(effects
+				(font
+					(size 1.27 1.27)
+				)
+				(justify left)
+			)
+		)
+		(property "Footprint" "Resistor_SMD:R_0603_1608Metric"
+			(at 133.35 136.398 90)
+			(effects
+				(font
+					(size 1.27 1.27)
+				)
+				(hide yes)
+			)
+		)
+		(property "Datasheet" "~"
+			(at 133.35 134.62 0)
+			(effects
+				(font
+					(size 1.27 1.27)
+				)
+				(hide yes)
+			)
+		)
+		(property "Description" "Resistor"
+			(at 133.35 134.62 0)
+			(effects
+				(font
+					(size 1.27 1.27)
+				)
+				(hide yes)
+			)
+		)
+		(pin "2"
+		)
+		(pin "1"
+		)
+		(instances
+			(project ""
+				(path "/566d9d78-0625-4273-b3cf-4edf1fc2bf65"
+					(reference "R10")
+					(unit 1)
+				)
+			)
+		)
+	)
+	(symbol
+		(lib_id "power:PWR_FLAG")
+		(at 165.1 120.65 0)
+		(unit 1)
+		(exclude_from_sim no)
+		(in_bom yes)
+		(on_board yes)
+		(dnp no)
+		(property "Reference" "#FLG03"
+			(at 165.1 118.745 0)
+			(effects
+				(font
+					(size 1.27 1.27)
+				)
+				(hide yes)
+			)
+		)
+		(property "Value" "PWR_FLAG"
+			(at 165.1 116.84 0)
+			(effects
+				(font
+					(size 1.27 1.27)
+				)
+			)
+		)
+		(property "Footprint" ""
+			(at 165.1 120.65 0)
+			(effects
+				(font
+					(size 1.27 1.27)
+				)
+				(hide yes)
+			)
+		)
+		(property "Datasheet" "~"
+			(at 165.1 120.65 0)
+			(effects
+				(font
+					(size 1.27 1.27)
+				)
+				(hide yes)
+			)
+		)
+		(property "Description" "Special symbol for telling ERC where power comes from"
+			(at 165.1 120.65 0)
+			(effects
+				(font
+					(size 1.27 1.27)
+				)
+				(hide yes)
+			)
+		)
+		(pin "1"
+		)
+		(instances
+			(project "clock-card"
+				(path "/566d9d78-0625-4273-b3cf-4edf1fc2bf65"
+					(reference "#FLG03")
+					(unit 1)
+				)
